File: EAGLE Board Designs/Main ECU/MainECU rev8.sch (EAGLE design)
At the start: 218 parts, among them J1 JUMPER, J2 JUMPER, J3 JUMPER, J4 JUMPER, J5 JUMPER, J6 JUMPER, J7 JUMPER, J8 JUMPER, P1 SOLDER_PAD, P2 SOLDER_PAD, Q1 P-CHANNEL_MOSFET_DMP3099L-7, Q12 P-CHANNEL_MOSFET_DMP3099L-7, X1 CONNECTOR-37, X2 CONNECTOR-4AUTOSPORT, X3 CONNECTOR-4NANO-FIT-VERTICAL-4, X4 CONNECTOR-4NANO-FIT-VERTICAL-4

Commit message: added BSPD schematic
Parts:
- added LED15: YELLOW, HyTechDevices:LED-0805
- added LED16: GREEN, HyTechDevices:LED-0805
- added LED2: RED, HyTechDevices:LED-0805
- added R67, R68: 270, HyTechDevices:RESISTOR0805-RES
- added R69: 200, HyTechDevices:RESISTOR0805-RES
- added U$14, U$15: TEST_POINT, HyTechDevices:TEST_POINT
Connections:
- new net N$64: LED2.C, R67.2
- new net N$76: LED15.C, R68.2
- new net N$77: LED16.C, R69.2
- new net READ_CHARGE: LED15.A, U$12.VINA-, U$12.VOUTA
- new net READ_FAULT: LED16.A, U$12.VINB-, U$12.VOUTB
- new net READ_SWITCH: LED2.A, U$6.4
- new net SIGNAL_BRAKE_FILT: C3.2, R12.2, R4.2, U$10.VINB+
- new net SIGNAL_CURRENT: R10.1, U$15.P$1
- new net SIGNAL_CURRENT_FILT: C2.2, R10.2, R7.1, U$10.VINA+
- net +12V: now also D2.C, R2.2, U$1.COIL-, U$3.3, U$3.4, U$3.COIL-
- net +5V: now also R13.2, R15.2, R4.1, R5.2, R7.2, U$10.VDD, U$12.VDD, U$4.VDD, U$5.5, U$6.5
- net GND: now also C1.2, C3.1, D2.A, D3.A, Q1.S, R1.1, R11.1, R14.1, R16.2, R67.1, R68.1, R69.1, R9.2, U$1.COIL+, U$10.VSS, U$12.VSS, U$4.VSS, U$5.3, U$6.3
- net N$1: now also D1.A, Q1.D, U$3.COIL+
- net N$13: now also C1.1, R3.1, R5.1, U$12.VINA+, U$4.VINA+
- net N$14: now also LED2.C, R8.1
- net N$15: now also LED1.C, R9.1
- net N$16: now also LED1.A, U$10.VOUTB, U$11.P$1, U$5.2, U$6.2
- net N$17: now also LED2.A, U$10.VOUTA, U$13.P$1, U$5.1, U$6.1
- net N$2: now also R3.2, U$5.4
- net N$3: now also D3.C, Q1.G, R16.1, U$4.VOUTA
- net N$5: now also R14.2, R15.1, U$10.VINA-
- net N$6: now also U$10.VINB-
- net N$7: now also R11.2, R13.1, U$4.VINA-
- net N$9: now also R1.2, R2.1, U$12.VINB+
- net SHUTDOWN_B: now also U$1.P
- net SHUTDOWN_C: now also U$1.S, U$3.6
- net SHUTDOWN_D: now also U$3.7
- net SIGNAL_BRAKE: now also R12.1, U$14.P$1
Other:
- note added: "Normally Open Relay -> FSAE EV5.1.6"
- moved on the sheet: D13, D15, D16, D17, D18, D5, D6, D7, LED1, LED17, LED18, LED3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
