File: EAGLE Board Designs/Main ECU/MainECU rev8.brd (EAGLE design)
At the start: 120.6 x 78.9 mm, 260 parts, among them J1 JUMPER, J2 JUMPER, J3 JUMPER, J4 JUMPER, J5 JUMPER, J6 JUMPER, J7 JUMPER, J8 JUMPER, P1 SOLDER_PAD, P2 SOLDER_PAD, Q1 P-CHANNEL_MOSFET_DMP3099L-7, Q12 P-CHANNEL_MOSFET_DMP3099L-7, X1 CONNECTOR-37, X2 CONNECTOR-4AUTOSPORT, X3 CONNECTOR-4NANO-FIT-VERTICAL-4, X4 CONNECTOR-4NANO-FIT-VERTICAL-4

Commit message: Added resistor values for the BSPD timing circuit.
Changed resistor from 330 -> 8200, added values on voltage divider (220, 330).
Parts:
- BSPD1:R11: value TBD -> 220
- BSPD1:R13: value TBD -> 330
- BSPD1:R3: value 330 -> 8200

Commit message: Verified that AND gate with drain and comparator function properly.
Note: resistor and capacitor values are subject to change; 100ms at present.
Parts:
- BSPD1:C1: value .47µ -> 47µ
- BSPD1:R11: value 220 -> 5.6K
- BSPD1:R13: value 330 -> 8.2K
- BSPD1:R3: value 8200 -> 220
- BSPD1:R5: value 680k -> 4.6K
Changed lines of the file:
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@@
 <element name="U$14" library="HyTechDevices" package="TEST_POINT" value="TEST_POINT" x="26.8224" y="-59.182" smashed="yes"/>
 <element name="U$15" library="HyTechDevices" package="TEST_POINT" value="TEST_POINT" x="30.1244" y="-59.182" smashed="yes"/>
-<element name="BSPD1:C1" library="HyTechDevices" package="0805" value=".47µ" x="-5.842" y="-66.04" smashed="yes">
+<element name="BSPD1:C1" library="HyTechDevices" package="0805" value="47µ" x="-5.842" y="-66.04" smashed="yes">
 <attribute name="NAME" x="-5.842" y="-65.3161" size="0.3048" layer="25" align="bottom-center"/>
 <attribute name="VALUE" x="-5.842" y="-66.7512" size="0.3048" layer="27" align="top-center"/>
@@
 <attribute name="VALUE" x="8.7884" y="-66.7512" size="0.3048" layer="27" align="top-center"/>
 </element>
-<element name="BSPD1:R3" library="HyTechDevices" package="0805" value="8200" x="12.446" y="-66.04" smashed="yes">
+<element name="BSPD1:R3" library="HyTechDevices" package="0805" value="220" x="12.446" y="-66.04" smashed="yes">
 <attribute name="NAME" x="12.446" y="-65.3161" size="0.3048" layer="25" align="bottom-center"/>
 <attribute name="VALUE" x="12.446" y="-66.7512" size="0.3048" layer="27" align="top-center"/>
@@
 <attribute name="VALUE" x="16.1036" y="-66.7512" size="0.3048" layer="27" align="top-center"/>
 </element>
-<element name="BSPD1:R5" library="HyTechDevices" package="0805" value="680k" x="19.7612" y="-66.04" smashed="yes">
+<element name="BSPD1:R5" library="HyTechDevices" package="0805" value="4.6K" x="19.7612" y="-66.04" smashed="yes">
 <attribute name="NAME" x="19.7612" y="-65.3161" size="0.3048" layer="25" align="bottom-center"/>
 <attribute name="VALUE" x="19.7612" y="-66.7512" size="0.3048" layer="27" align="top-center"/>
@@
 <attribute name="NAME" x="16.5862" y="-60.5504" size="0.762" layer="25" font="vector" rot="R270" align="center"/>
 </element>
-<element name="BSPD1:R11" library="HyTechDevices" package="0805" value="220" x="-5.842" y="-70.9676" smashed="yes">
+<element name="BSPD1:R11" library="HyTechDevices" package="0805" value="5.6K" x="-5.842" y="-70.9676" smashed="yes">
 <attribute name="NAME" x="-5.842" y="-70.2437" size="0.3048" layer="25" align="bottom-center"/>
 <attribute name="VALUE" x="-5.842" y="-71.6788" size="0.3048" layer="27" align="top-center"/>
 </element>
-<element name="BSPD1:R13" library="HyTechDevices" package="0805" value="330" x="-5.842" y="-73.4314" smashed="yes">
+<element name="BSPD1:R13" library="HyTechDevices" package="0805" value="8.2K" x="-5.842" y="-73.4314" smashed="yes">
 <attribute name="NAME" x="-5.842" y="-72.7075" size="0.3048" layer="25" align="bottom-center"/>
 <attribute name="VALUE" x="-5.842" y="-74.1426" size="0.3048" layer="27" align="top-center"/>
