File: EAGLE Board Designs/Main ECU/BSPD rev11.brd (EAGLE design)
At the start: 87.6 x 100 mm, 54 parts, among them Q1 P-CHANNEL_MOSFET_DMP3099L-7, U11 SN74AHC1G09, U17 OPA990IDBVR, U19 OPA990IDBVR, U28 OPA990IDBVR, U29 OPA990IDBVR, U6 OPA990IDBVR, X1 CONNECTOR-4NANO-FIT-VERTICAL-4, X2 CONNECTOR-4NANO-FIT-VERTICAL-4

Commit message: I just added a cap sorry
Parts:
- added C1: 0.1uF, HyTechDevices:0603-CAP
Connections:
- net +12V: now also C1.2
- net GND: now also C1.1
Changed lines of the file:
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@@
 <attribute name="NAME" x="27.305" y="87.63" size="0.8128" layer="25"/>
+</element>
+<element name="C1" library="HyTechDevices" package="0603-CAP" value="0.1uF" x="2.54" y="-2.54" smashed="yes">
+<attribute name="NAME" x="1.651" y="-1.778" size="0.8128" layer="25" font="vector"/>
 </element>
 </elements>
@@
 <contactref element="R6" pad="1"/>
 <contactref element="R8" pad="1"/>
-<wire x1="46.99" y1="69" x2="50.8" y2="77.55" width="0" layer="19" extent="1-1"/>
-<wire x1="49.53" y1="70.27" x2="46.99" y2="69" width="0" layer="19" extent="1-1"/>
-<wire x1="40.56" y1="81.6" x2="46.99" y2="69" width="0" layer="19" extent="1-1"/>
+<contactref element="C1" pad="1"/>
+<wire x1="49.53" y1="70.27" x2="50.8" y2="77.55" width="0" layer="19" extent="1-1"/>
+<wire x1="46.99" y1="69" x2="49.53" y2="70.27" width="0" layer="19" extent="1-1"/>
+<wire x1="55.03" y1="68.58" x2="49.53" y2="70.27" width="0" layer="19" extent="1-1"/>
+<wire x1="53.32" y1="59.69" x2="55.03" y2="68.58" width="0" layer="19" extent="1-1"/>
+<wire x1="40.56" y1="81.6" x2="50.8" y2="77.55" width="0" layer="19" extent="1-1"/>
 <wire x1="41.06" y1="86.36" x2="40.56" y2="81.6" width="0" layer="19" extent="1-1"/>
-<wire x1="35.56" y1="80.43" x2="41.06" y2="86.36" width="0" layer="19" extent="1-1"/>
-<wire x1="36.83" y1="87.71" x2="35.56" y2="80.43" width="0" layer="19" extent="1-1"/>
+<wire x1="36.83" y1="87.71" x2="41.06" y2="86.36" width="0" layer="19" extent="1-1"/>
 <wire x1="33.02" y1="85.51" x2="36.83" y2="87.71" width="0" layer="19" extent="1-1"/>
+<wire x1="35.56" y1="80.43" x2="40.56" y2="81.6" width="0" layer="19" extent="1-1"/>
 <wire x1="27.52" y1="87.63" x2="33.02" y2="85.51" width="0" layer="19" extent="1-1"/>
 <wire x1="21.59" y1="90.25" x2="27.52" y2="87.63" width="0" layer="19" extent="1-1"/>
-<wire x1="21.59" y1="82.97" x2="21.59" y2="90.25" width="0" layer="19" extent="1-1"/>
-<wire x1="16.51" y1="73.74" x2="21.59" y2="82.97" width="0" layer="19" extent="1-1"/>
-<wire x1="22.44" y1="71.12" x2="16.51" y2="73.74" width="0" layer="19" extent="1-1"/>
-<wire x1="29.21" y1="70.27" x2="22.44" y2="71.12" width="0" layer="19" extent="1-1"/>
-<wire x1="33.02" y1="72.47" x2="29.21" y2="70.27" width="0" layer="19" extent="1-1"/>
-<wire x1="31.75" y1="65.19" x2="33.02" y2="72.47" width="0" layer="19" extent="1-1"/>
-<wire x1="16.51" y1="66.46" x2="16.51" y2="73.74" width="0" layer="19" extent="1-1"/>
-<wire x1="13.97" y1="67.73" x2="16.51" y2="66.46" width="0" layer="19" extent="1-1"/>
-<wire x1="19.05" y1="84.24" x2="21.59" y2="82.97" width="0" layer="19" extent="1-1"/>
+<wire x1="19.05" y1="84.24" x2="21.59" y2="90.25" width="0" layer="19" extent="1-1"/>
 <wire x1="16.51" y1="84.24" x2="19.05" y2="84.24" width="0" layer="19" extent="1-1"/>
-<wire x1="6.67" y1="85.36" x2="16.51" y2="84.24" width="0" layer="19" extent="1-1"/>
-<wire x1="7.62" y1="81.26" x2="6.67" y2="85.36" width="0" layer="19" extent="1-1"/>
-<wire x1="7.35" y1="72.71" x2="7.62" y2="81.26" width="0" layer="19" extent="1-1"/>
-<wire x1="11.43" y1="67.73" x2="7.35" y2="72.71" width="0" layer="19" extent="1-1"/>
-<wire x1="55.03" y1="68.58" x2="11.43" y2="67.73" width="0" layer="19" extent="1-1"/>
-<wire x1="44.45" y1="52.49" x2="55.03" y2="68.58" width="0" layer="19" extent="1-1"/>
-<wire x1="26.67" y1="52.49" x2="44.45" y2="52.49" width="0" layer="19" extent="1-1"/>
-<wire x1="35.56" y1="55.88" x2="44.45" y2="52.49" width="0" layer="19" extent="1-1"/>
-<wire x1="53.32" y1="59.69" x2="35.56" y2="55.88" width="0" layer="19" extent="1-1"/>
+<wire x1="21.59" y1="82.97" x2="19.05" y2="84.24" width="0" layer="19" extent="1-1"/>
+<wire x1="33.02" y1="72.47" x2="35.56" y2="80.43" width="0" layer="19" extent="1-1"/>
+<wire x1="29.21" y1="70.27" x2="33.02" y2="72.47" width="0" layer="19" extent="1-1"/>
+<wire x1="31.75" y1="65.19" x2="29.21" y2="70.27" width="0" layer="19" extent="1-1"/>
+<wire x1="22.44" y1="71.12" x2="29.21" y2="70.27" width="0" layer="19" extent="1-1"/>
+<wire x1="16.51" y1="73.74" x2="22.44" y2="71.12" width="0" layer="19" extent="1-1"/>
+<wire x1="13.97" y1="67.73" x2="16.51" y2="73.74" width="0" layer="19" extent="1-1"/>
+<wire x1="11.43" y1="67.73" x2="13.97" y2="67.73" width="0" layer="19" extent="1-1"/>
+<wire x1="16.51" y1="66.46" x2="13.97" y2="67.73" width="0" layer="19" extent="1-1"/>
+<wire x1="7.35" y1="72.71" x2="11.43" y2="67.73" width="0" layer="19" extent="1-1"/>
+<wire x1="7.62" y1="81.26" x2="7.35" y2="72.71" width="0" layer="19" extent="1-1"/>
+<wire x1="6.67" y1="85.36" x2="7.62" y2="81.26" width="0" layer="19" extent="1-1"/>
+<wire x1="35.56" y1="55.88" x2="31.75" y2="65.19" width="0" layer="19" extent="1-1"/>
+<wire x1="44.45" y1="52.49" x2="35.56" y2="55.88" width="0" layer="19" extent="1-1"/>
+<wire x1="26.67" y1="52.49" x2="35.56" y2="55.88" width="0" layer="19" extent="1-1"/>
+<wire x1="1.69" y1="-2.54" x2="26.67" y2="52.49" width="0" layer="19" extent="1-1"/>
 </signal>
 <signal name="+12V">
@@
 <contactref element="REG2" pad="1"/>
 <contactref element="C105" pad="2"/>
-<wire x1="51.75" y1="74.85" x2="7.62" y2="78.76" width="0" layer="19" extent="1-1"/>
-<wire x1="57.47" y1="77.2" x2="51.75" y2="74.85" width="0" layer="19" extent="1-1"/>
-<wire x1="58.42" y1="82.28" x2="57.47" y2="77.2" width="0" layer="19" extent="1-1"/>
-<wire x1="63.08" y1="78.74" x2="58.42" y2="82.28" width="0" layer="19" extent="1-1"/>
-<wire x1="26.67" y1="54.19" x2="63.08" y2="78.74" width="0" layer="19" extent="1-1"/>
-<wire x1="50.82" y1="59.69" x2="57.47" y2="77.2" width="0" layer="19" extent="1-1"/>
+<contactref element="C1" pad="2"/>
+<wire x1="57.47" y1="77.2" x2="58.42" y2="82.28" width="0" layer="19" extent="1-1"/>
+<wire x1="63.08" y1="78.74" x2="57.47" y2="77.2" width="0" layer="19" extent="1-1"/>
+<wire x1="51.75" y1="74.85" x2="57.47" y2="77.2" width="0" layer="19" extent="1-1"/>
+<wire x1="50.82" y1="59.69" x2="51.75" y2="74.85" width="0" layer="19" extent="1-1"/>
 <wire x1="33.02" y1="55.88" x2="50.82" y2="59.69" width="0" layer="19" extent="1-1"/>
+<wire x1="26.67" y1="54.19" x2="33.02" y2="55.88" width="0" layer="19" extent="1-1"/>
+<wire x1="7.62" y1="78.76" x2="26.67" y2="54.19" width="0" layer="19" extent="1-1"/>
+<wire x1="3.39" y1="-2.54" x2="26.67" y2="54.19" width="0" layer="19" extent="1-1"/>
 </signal>
 <signal name="+5V">
