File: EAGLE Board Designs/Data Acquisition Boards/Wheel Speend Sensor/Wheel Speed Sensor rev1.4.brd (EAGLE design)
At the start: 50.8 x 56.8 mm, 16 parts, among them X1 Sensor 1, X2 Sensor 2, X4 CONNECTOR-4, X5 CONNECTOR-4

Commit message: Changed capacitor value
Parts:
- C6: value 1uF -> .1 uF
Changed lines of the file:
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@@
 <attribute name="VALUE" x="-7.366" y="-12.954" size="0.4064" layer="27"/>
 </element>
-<element name="C6" library="HyTechDevices" package="CAP-PTH-5MM" value="1uF" x="-6.35" y="-13.97" smashed="yes">
+<element name="C6" library="HyTechDevices" package="CAP-PTH-5MM" value=".1 uF" x="-6.35" y="-13.97" smashed="yes">
 <attribute name="NAME" x="-7.112" y="-12.7" size="0.4064" layer="25"/>
 <attribute name="VALUE" x="-7.366" y="-15.494" size="0.4064" layer="27"/>
