File: EAGLE Board Designs/Data Acquisition Boards/Strain Gauge/strain gage 10V loadcell test rev1.sch (EAGLE design)
At the start: 24 parts, among them Q1 MMBT4403, U1 HX711, X1 CONNECTOR-6, X4 CONNECTOR-4, X5 CONNECTOR-4

Commit message: Cleaned up file naming
Parts:
- added C12, C16, C17: 0.1uF, HyTechDevices:CAP0805
- added C13: 1uF, HyTechDevices:CAP0805
- added C14: .1uF, HyTechDevices:CAP0805
- added C18: 10uF, HyTechDevices:CAP0805
- added L2: 3.3uH, SparkFun-Passives:INDUCTOR0805-IND
- added Q2: MMBT4403, SparkFun-DiscreteSemi:TRANSISTOR_PNPMMBT4403
- added R10, R11, R9: (no value), HyTechDevices:RESISTORAXIAL-0.3
- added R12: 20k, HyTechDevices:RESISTOR0805-RES
- added R13: 8.2k, HyTechDevices:RESISTORAXIAL-0.3
- added R14, R15: 100, HyTechDevices:RESISTORAXIAL-0.3
- added R16, R7: 6800, HyTechDevices:RESISTORAXIAL-0.3
- added R17, R8: 3300, HyTechDevices:RESISTORAXIAL-0.3
- added R5: 200, HyTechDevices:RESISTOR0805-RES
- added R6: 1000, HyTechDevices:RESISTORAXIAL-0.3
- added U$2: CPC1002N, HyTechDevices:CPC1002N
- added U2: HX711, Testing:HX711HX711
- added X2: CONNECTOR-2, HyTechDevices:CONNECTOR-2
- C1, C2, C3, C4: device SparkFun-Capacitors:0.1UF-25V-5%(0603) -> HyTechDevices:CAP0805
- C5: value 0.1uF -> 10uF; device SparkFun-Capacitors:0.1UF-25V-5%(0603) -> HyTechDevices:CAP0805
- C6: value 10uF -> 0.1uF; device SparkFun-Capacitors:10UF50V20%(1210) -> HyTechDevices:CAP0805
- C7: device SparkFun-Capacitors:10UF50V20%(1210) -> HyTechDevices:CAP0805
- R1: device SparkFun-Resistors:20KOHM1/10W1%(0603) -> HyTechDevices:RESISTOR0805-RES
- R2: value 8.2K -> 8.2k; device SparkFun-Resistors:8.2KOHM-1/10W-5%(0603) -> HyTechDevices:RESISTORAXIAL-0.3
- R3, R4: device SparkFun-Resistors:100OHM-1/10W-1%(0603) -> HyTechDevices:RESISTORAXIAL-0.3
Connections:
- removed net VDD: C4.1
- new net A+2: R3.1, R9.2, X2-2.S
- new net A-2: R10.1, R11.1, R4.1
- new net AVDD2: C12.1, C7.1, L2.1, R11.2, X2-1.S
- new net N$1: Q2.B, U2.BASE
- new net N$10: C1.2, U2.VBG
- new net N$11: L2.2, Q2.C, R1.2, U2.AVDD
- new net N$12: C2.2, R3.2, U2.INA+
- new net N$13: R16.2, X1-4.S
- new net N$14: C13.2, C14.2, U$2.DC-, X1-1.S
- new net N$15: R5.2, R6.1, U$2.DC+
- new net N$16: R7.2, X1-3.S
- new net N$8: C2.1, R4.2, U2.INA-
- new net N$9: R1.1, R2.2, U2.VFB
- net A+: now also R15.1, R16.1, R17.2; no longer R4.1, X1-4.S
- net A-: now also R14.1, R7.1, R8.2; no longer R3.1, X1-3.S
- net AVDD: now also C4.1, C5.1, U$2.CONTROL+; no longer C3.1, C7.1, X1-1.S
- net DAT2: now also U2.DOUT
- net GND: now also C1.1, C12.2, C13.1, C14.1, C16.2, C17.2, C18.2, C6.1, R10.2, R13.1, R17.1, R6.2, R8.1, R9.1, U$2.CONTROL-, U2.AGND, U2.INB+, U2.INB-, U2.RATE, U2.XI; no longer C2.1, C3.2, C6.2
- net N$2: now also C3.1, R14.2; no longer C1.1, R3.2
- net N$3: now also C3.2, R15.2; no longer C1.2, R4.2
- net N$5: now also R12.2; no longer R1.2
- net N$6: now also R12.1, R13.2; no longer R1.1, R2.2
- net N$7: now also C6.2; no longer C2.2
- net SCK2: now also U2.PD_SCK
- net VCC: now also C16.1, C17.1, C18.1, Q2.E, U2.DVDD, U2.VSUP; no longer C5.1, C6.1
- net VIN: now also R5.1
Other:
- note added: "teensy 4.0"
- moved on the sheet: C1, C2, C3, C4, C5, C6, C7, R1, R2, R3, R4
