File: EAGLE Board Designs/Panelized Orders/2019-12-15/Charger Controller, HV Board, TSAL, Strain Guage, and ADIS Practice.brd (EAGLE design)
At the start: 266.1 x 146.3 mm, 344 parts, among them IC1 KX124-1051, IC2 KX124-1051, IC3 KX124-1051, IC4 KX124-1051, IC5 KX124-1051, IC6 KX124-1051, IC7 KX124-1051, IC8 KX124-1051, IC9 KX124-1051, J1 JUMPER.1, J2 JUMPER.1, J3 JUMPER.1, J4 JUMPER.1, Q2 DMG3406L, Q3 DMG3406L, U1 OPA2172, U10 STWD100, U11 HM2102NLT, U12 MCP3208SOIC, U13 TXB0104TSSOP, U14 MCP6542SOIC, U16 UCC21520A, U17 LR8, U18 CDSOT23-T24CAN-Q, U19 LTC6082CGNPBF, U2 OKI-78SR-5, U20 LTC6082CGNPBF, U3 MAX7480, U4 MAX7480, U5 MAX7480, U6 MAX7480, U7 MCP2551, U8 SN74LVC1G08, U9 LTC6820, X2 CONNECTOR-4, X3 CONNECTOR-4NANO-FIT-VERTICAL-4

Commit message: Added fiducials and adjusted final spacing
Parts:
- moved C3 19.1 mm to (64.5, 36.3)
- moved C4 19.1 mm to (64.5, 41.4)
- moved R15 19.1 mm to (50.5, 37.6)
- moved REG 19.1 mm to (72.1, 40.2)
- moved STATUS 19.1 mm to (50.5, 40.2)
- moved U$1 19.1 mm to (54.3, 66.8)
- moved U$5 19.1 mm to (59.4, 45.2)
- moved D6 19.1 mm to (30.2, 74.4)
- moved POWERTAIL 19.1 mm to (30.2, 26.2)
- moved R11 19.1 mm to (30.2, 63.0)
- moved R12 19.1 mm to (30.2, 57.9)
- moved R2 19.1 mm to (30.2, 71.9)
- moved S1 19.1 mm to (18.7, 38.9)
- moved U$2 19.1 mm to (30.2, 37.6)
- moved 5ABOARDFUSE 19.1 mm to (13.7, 49.0)
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Other:
- board size 266.1 x 146.3 mm -> 247.3 x 142.9 mm
