File: EAGLE Board Designs/BMS/BMS Cell Charging Adapter/BMS Cell Charging Adapter rev2.brd (EAGLE design)
At the start: 108 x 298.8 mm, 21 parts, among them X1 CONNECTOR-10, X2 CONNECTOR-10

Commit message: Changed the locations of the pads on the charger controller pcb layout
Parts:
- moved CELL1 16.2 mm to (29.0, 21.2)
- moved CELL0 14.0 mm to (79.0, 18.7)
- moved CELL2 13.4 mm to (79.0, 43.3)
- moved CELL3 12.3 mm to (29.0, 45.9)
- moved CELL4 11.4 mm to (79.0, 68.0)
- moved CELL5 10.3 mm to (29.0, 70.5)
- moved CELL6 9.40 mm to (79.0, 92.6)
- moved CELL7 8.32 mm to (29.0, 95.1)
- moved CELL8 7.40 mm to (79.0, 117.2)
- moved CELL9 6.31 mm to (29.0, 119.8)
- moved CELL10 5.39 mm to (79.0, 141.9)
- moved CELL11 4.30 mm to (29.0, 144.4)
- moved CELL12 3.38 mm to (79.0, 166.5)
- moved CELL18 3.34 mm to (79.0, 240.9)
- moved CELL13 2.30 mm to (29.0, 169.0)
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Routing:
- net CELL1: track 23.7 -> 39.9 mm
- net CELL2: track 61.0 -> 74.5 mm
- net CELL0: track 43.3 -> 56.7 mm
- net CELL3: track 55.6 -> 68.0 mm
- net CELL4: track 87.3 -> 99.1 mm
- net CELL5: track 90.3 -> 100.6 mm
- net CELL6: track 136.3 -> 146.2 mm
- net CELL7: track 131.2 -> 140.4 mm
- net CELL8: track 156.8 -> 164.9 mm
- net CELL10: track 136.4 -> 131.3 mm
- net CELL12: track 108.7 -> 105.3 mm
- net CELL11: track 123.9 -> 121.1 mm
- net CELL18: track 53.0 -> 55.7 mm
- net CELL13: track 93.8 -> 91.5 mm
- net CELL17: track 49.9 -> 51.7 mm
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
Commit message: changed the locations of the pads in the Cell Charging adapter board
Parts:
- moved CELL1 9.61 mm to (38.6, 21.2)
- moved CELL11 9.61 mm to (38.6, 144.4)
- moved CELL13 9.61 mm to (38.6, 169.0)
- moved CELL15 9.61 mm to (38.6, 193.7)
- moved CELL17 9.61 mm to (38.6, 218.3)
- moved CELL3 9.61 mm to (38.6, 45.9)
- moved CELL5 9.61 mm to (38.6, 70.5)
- moved CELL7 9.61 mm to (38.6, 95.1)
- moved CELL9 9.61 mm to (38.6, 119.8)
Routing:
- net CELL15: track 83.5 -> 100.4 mm
- net CELL13: track 91.5 -> 101.5 mm
- net CELL9: track 363.7 -> 354.0 mm
- net CELL5: track 100.6 -> 108.7 mm
- net CELL11: track 121.1 -> 125.6 mm
- net CELL3: track 68.0 -> 71.0 mm
- net CELL1: track 39.9 -> 42.5 mm
- net CELL17: track 51.7 -> 50.4 mm
- net CELL7: track 140.4 -> 139.4 mm

Commit message: Made changes to the charger adapter rev2 board
Parts:
- CELL0, CELL1, CELL10, CELL11, CELL12, CELL13, CELL14, CELL15, CELL16, CELL17, CELL18, CELL2, CELL3, CELL4, CELL5, CELL6, CELL7, CELL8, CELL9: value BATTERY_SPRING -> BATTERY_SPRING_KEYSTONE5222; device HyTechDevices:KEYSTONE5203 -> HyTechDevices:KEYSTONE5222
Routing:
- net CELL9: track 354.0 -> 370.2 mm
- net CELL15: track 100.4 -> 88.6 mm
- net CELL5: track 108.7 -> 99.3 mm
- net CELL11: track 125.6 -> 117.7 mm
- net CELL3: track 71.0 -> 64.0 mm
- net CELL1: track 42.5 -> 35.9 mm
- net CELL17: track 50.4 -> 56.7 mm
- net CELL13: track 101.5 -> 95.5 mm
- net CELL10: track 131.3 -> 136.9 mm
- net CELL4: track 99.1 -> 104.2 mm
- net CELL7: track 139.4 -> 144.0 mm
- net CELL6: track 146.2 -> 149.5 mm
- net CELL8: track 164.9 -> 168.1 mm
