File: EAGLE Board Designs/BMS/BMS Enerdel Adapter/BMS Enerdel Adapter rev4.brd (EAGLE design)
At the start: 108 x 331.4 mm, 27 parts

Commit message: Finished the enerdal adapter rev 5 of the pcb design
Parts:
- CELL0, CELL1, CELL10, CELL11, CELL12, CELL13, CELL14, CELL15, CELL16, CELL17, CELL18, CELL2, CELL3, CELL4, CELL5, CELL6, CELL7, CELL8, CELL9: value BATTERY_SPRING -> BATTERY_SPRING_KEYSTONE5222; device HyTechDevices:KEYSTONE5203 -> HyTechDevices:KEYSTONE5222
- moved CELL17 11.7 mm to (33.5, 209.3)
- moved CELL16 10.9 mm to (73.9, 206.8)
- moved CELL15 9.85 mm to (33.5, 184.7)
- moved CELL14 9.20 mm to (73.9, 182.1)
- moved CELL13 8.11 mm to (33.5, 160.0)
- moved CELL1 7.83 mm to (33.5, 11.4)
- moved CELL12 7.60 mm to (73.9, 157.5)
- moved CELL2 6.56 mm to (73.9, 34.0)
- moved CELL11 6.55 mm to (33.5, 135.4)
- moved CELL10 6.40 mm to (73.9, 132.6)
- moved CELL18 6.25 mm to (77.5, 234.9)
- moved CELL4 5.52 mm to (73.9, 58.7)
- moved CELL3 5.46 mm to (33.5, 36.6)
- moved CELL8 5.42 mm to (73.9, 108.0)
- moved CELL9 5.42 mm to (33.5, 110.5)
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Routing:
- net A18-B24: track 193.5 -> 206.1 mm
- net A16-B22: track 222.0 -> 232.6 mm
- net A14-B20: track 197.0 -> 205.6 mm
- net A8-B14: track 397.5 -> 404.2 mm
- net A3-B9: track 163.5 -> 170.0 mm
- net A7-B13: track 413.5 -> 419.6 mm
- net A4-B10: track 153.5 -> 159.3 mm
- net A15-B21: track 243.7 -> 249.3 mm
- net A11-B17: track 407.1 -> 412.2 mm
- net A6-B12: track 182.9 -> 187.9 mm
- net A17-B23: track 202.6 -> 207.5 mm
- net A5-B11: track 179.0 -> 183.4 mm
- net A19-B25: track 138.5 -> 142.8 mm
- net A10-B16: track 410.4 -> 414.6 mm
- net A1-B7: track 117.2 -> 119.1 mm
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Other:
- outline, holes or cut-outs redrawn
