File: EAGLE Board Designs/BMS/BMS Enerdel Adapter/BMS Enerdel Adapter rev4.brd (EAGLE design)
At the start: 108 x 331.4 mm, 27 parts

Commit message: Updated the Enerdal_Adapter
Routing:
- net A18-B24: track 206.1 -> 207.5 mm
Changed lines of the file:
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@@
 <wire x1="33.528" y1="209.296" x2="29" y2="213.824" width="0.4064" layer="1"/>
 <wire x1="29" y1="213.824" x2="29" y2="249.98" width="0.4064" layer="1"/>
+<wire x1="33.528" y1="209.296" x2="34.544" y2="208.28" width="0.4064" layer="1"/>
 </signal>
 <signal name="A19-B25">

Commit message: Made file changes so that the files were correctly named
Parts:
- CELL0, CELL1, CELL10, CELL11, CELL12, CELL13, CELL14, CELL15, CELL16, CELL17, CELL18, CELL2, CELL3, CELL4, CELL5, CELL6, CELL7, CELL8, CELL9: value BATTERY_SPRING_KEYSTONE5222 -> BATTERY_SPRING; device HyTechDevices:KEYSTONE5222 -> HyTechDevices:KEYSTONE5203
- moved CELL17 11.7 mm to (29.0, 220.1)
- moved CELL16 10.9 mm to (79.0, 216.4)
- moved CELL15 9.85 mm to (29.0, 193.4)
- moved CELL14 9.20 mm to (79.0, 189.8)
- moved CELL13 8.11 mm to (29.0, 166.8)
- moved CELL1 7.83 mm to (29.0, 5.04)
- moved CELL12 7.60 mm to (79.0, 163.1)
- moved CELL2 6.56 mm to (79.0, 29.9)
- moved CELL11 6.55 mm to (29.0, 140.1)
- moved CELL10 6.40 mm to (79.0, 136.5)
- moved CELL18 6.25 mm to (75.7, 240.9)
- moved CELL4 5.52 mm to (79.0, 56.5)
- moved CELL3 5.46 mm to (29.0, 33.5)
- moved CELL8 5.42 mm to (79.0, 109.8)
- moved CELL9 5.42 mm to (29.0, 113.5)
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Routing:
- net A18-B24: track 207.5 -> 193.5 mm
- net A16-B22: track 232.6 -> 222.0 mm
- net A14-B20: track 205.6 -> 197.0 mm
- net A8-B14: track 404.2 -> 397.5 mm
- net A3-B9: track 170.0 -> 163.5 mm
- net A7-B13: track 419.6 -> 413.5 mm
- net A4-B10: track 159.3 -> 153.5 mm
- net A15-B21: track 249.3 -> 243.7 mm
- net A11-B17: track 412.2 -> 407.1 mm
- net A6-B12: track 187.9 -> 182.9 mm
- net A17-B23: track 207.5 -> 202.6 mm
- net A5-B11: track 183.4 -> 179.0 mm
- net A19-B25: track 142.8 -> 138.5 mm
- net A10-B16: track 414.6 -> 410.4 mm
- net A1-B7: track 119.1 -> 117.2 mm
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Other:
- outline, holes or cut-outs redrawn
