File: EAGLE Board Designs/BMS/BMS Enerdel Adapter/BMS Enerdel Adapter rev4.sch (EAGLE design)
At the start: 27 parts

Commit message: Finished the enerdal adapter rev 5 of the pcb design
Parts:
- CELL0, CELL1, CELL10, CELL11, CELL12, CELL13, CELL14, CELL15, CELL16, CELL17, CELL18, CELL2, CELL3, CELL4, CELL5, CELL6, CELL7, CELL8, CELL9: value BATTERY_SPRING -> BATTERY_SPRING_KEYSTONE5222; device HyTechDevices:BATTERY_SPRING -> HyTechDevices:BATTERY_SPRING_KEYSTONE5222
Changed lines of the file:
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@@
 <?xml version="1.0" encoding="utf-8"?>
 <!DOCTYPE eagle SYSTEM "eagle.dtd">
-<eagle version="9.2.2">
+<eagle version="9.6.2">
 <drawing>
 <settings>
@@
 <layer number="154" name="FabDoc2" color="7" fill="1" visible="yes" active="yes"/>
 <layer number="155" name="FabDoc3" color="7" fill="1" visible="yes" active="yes"/>
+<layer number="156" name="HVSpacing" color="12" fill="1" visible="no" active="yes"/>
 <layer number="191" name="mNets" color="7" fill="1" visible="yes" active="yes"/>
 <layer number="192" name="mBusses" color="7" fill="1" visible="yes" active="yes"/>
@@
 </modules>
 <parts>
-<part name="CELL9" library="HyTechDevices" deviceset="BATTERY_SPRING" device="" value="BATTERY_SPRING"/>
-<part name="CELL8" library="HyTechDevices" deviceset="BATTERY_SPRING" device="" value="BATTERY_SPRING"/>
-<part name="CELL7" library="HyTechDevices" deviceset="BATTERY_SPRING" device="" value="BATTERY_SPRING"/>
-<part name="CELL6" library="HyTechDevices" deviceset="BATTERY_SPRING" device="" value="BATTERY_SPRING"/>
-<part name="CELL4" library="HyTechDevices" deviceset="BATTERY_SPRING" device="" value="BATTERY_SPRING"/>
-<part name="CELL5" library="HyTechDevices" deviceset="BATTERY_SPRING" device="" value="BATTERY_SPRING"/>
-<part name="CELL3" library="HyTechDevices" deviceset="BATTERY_SPRING" device="" value="BATTERY_SPRING"/>
-<part name="CELL2" library="HyTechDevices" deviceset="BATTERY_SPRING" device="" value="BATTERY_SPRING"/>
-<part name="CELL1" library="HyTechDevices" deviceset="BATTERY_SPRING" device="" value="BATTERY_SPRING"/>
-<part name="CELL0" library="HyTechDevices" deviceset="BATTERY_SPRING" device="" value="BATTERY_SPRING"/>
-<part name="CELL18" library="HyTechDevices" deviceset="BATTERY_SPRING" device="" value="BATTERY_SPRING"/>
-<part name="CELL17" library="HyTechDevices" deviceset="BATTERY_SPRING" device="" value="BATTERY_SPRING"/>
-<part name="CELL16" library="HyTechDevices" deviceset="BATTERY_SPRING" device="" value="BATTERY_SPRING"/>
-<part name="CELL15" library="HyTechDevices" deviceset="BATTERY_SPRING" device="" value="BATTERY_SPRING"/>
-<part name="CELL13" library="HyTechDevices" deviceset="BATTERY_SPRING" device="" value="BATTERY_SPRING"/>
-<part name="CELL14" library="HyTechDevices" deviceset="BATTERY_SPRING" device="" value="BATTERY_SPRING"/>
-<part name="CELL12" library="HyTechDevices" deviceset="BATTERY_SPRING" device="" value="BATTERY_SPRING"/>
-<part name="CELL11" library="HyTechDevices" deviceset="BATTERY_SPRING" device="" value="BATTERY_SPRING"/>
-<part name="CELL10" library="HyTechDevices" deviceset="BATTERY_SPRING" device="" value="BATTERY_SPRING"/>
+<part name="CELL9" library="HyTechDevices" deviceset="BATTERY_SPRING" device="_KEYSTONE5222" value="BATTERY_SPRING_KEYSTONE5222"/>
+<part name="CELL8" library="HyTechDevices" deviceset="BATTERY_SPRING" device="_KEYSTONE5222" value="BATTERY_SPRING_KEYSTONE5222"/>
+<part name="CELL7" library="HyTechDevices" deviceset="BATTERY_SPRING" device="_KEYSTONE5222" value="BATTERY_SPRING_KEYSTONE5222"/>
+<part name="CELL6" library="HyTechDevices" deviceset="BATTERY_SPRING" device="_KEYSTONE5222" value="BATTERY_SPRING_KEYSTONE5222"/>
+<part name="CELL4" library="HyTechDevices" deviceset="BATTERY_SPRING" device="_KEYSTONE5222" value="BATTERY_SPRING_KEYSTONE5222"/>
+<part name="CELL5" library="HyTechDevices" deviceset="BATTERY_SPRING" device="_KEYSTONE5222" value="BATTERY_SPRING_KEYSTONE5222"/>
+<part name="CELL3" library="HyTechDevices" deviceset="BATTERY_SPRING" device="_KEYSTONE5222" value="BATTERY_SPRING_KEYSTONE5222"/>
+<part name="CELL2" library="HyTechDevices" deviceset="BATTERY_SPRING" device="_KEYSTONE5222" value="BATTERY_SPRING_KEYSTONE5222"/>
+<part name="CELL1" library="HyTechDevices" deviceset="BATTERY_SPRING" device="_KEYSTONE5222" value="BATTERY_SPRING_KEYSTONE5222"/>
+<part name="CELL0" library="HyTechDevices" deviceset="BATTERY_SPRING" device="_KEYSTONE5222" value="BATTERY_SPRING_KEYSTONE5222"/>
+<part name="CELL18" library="HyTechDevices" deviceset="BATTERY_SPRING" device="_KEYSTONE5222" value="BATTERY_SPRING_KEYSTONE5222"/>
+<part name="CELL17" library="HyTechDevices" deviceset="BATTERY_SPRING" device="_KEYSTONE5222" value="BATTERY_SPRING_KEYSTONE5222"/>
+<part name="CELL16" library="HyTechDevices" deviceset="BATTERY_SPRING" device="_KEYSTONE5222" value="BATTERY_SPRING_KEYSTONE5222"/>
+<part name="CELL15" library="HyTechDevices" deviceset="BATTERY_SPRING" device="_KEYSTONE5222" value="BATTERY_SPRING_KEYSTONE5222"/>
+<part name="CELL13" library="HyTechDevices" deviceset="BATTERY_SPRING" device="_KEYSTONE5222" value="BATTERY_SPRING_KEYSTONE5222"/>
+<part name="CELL14" library="HyTechDevices" deviceset="BATTERY_SPRING" device="_KEYSTONE5222" value="BATTERY_SPRING_KEYSTONE5222"/>
+<part name="CELL12" library="HyTechDevices" deviceset="BATTERY_SPRING" device="_KEYSTONE5222" value="BATTERY_SPRING_KEYSTONE5222"/>
+<part name="CELL11" library="HyTechDevices" deviceset="BATTERY_SPRING" device="_KEYSTONE5222" value="BATTERY_SPRING_KEYSTONE5222"/>
+<part name="CELL10" library="HyTechDevices" deviceset="BATTERY_SPRING" device="_KEYSTONE5222" value="BATTERY_SPRING_KEYSTONE5222"/>
 <part name="A_LOWER_OUTPUT" library="HyTechDevices" deviceset="CONNECTOR-14" device=""/>
 <part name="A_LOWER_INPUT" library="HyTechDevices" deviceset="CONNECTOR-14" device=""/>

Commit message: Made file changes so that the files were correctly named
Parts:
- CELL0, CELL1, CELL10, CELL11, CELL12, CELL13, CELL14, CELL15, CELL16, CELL17, CELL18, CELL2, CELL3, CELL4, CELL5, CELL6, CELL7, CELL8, CELL9: value BATTERY_SPRING_KEYSTONE5222 -> BATTERY_SPRING; device HyTechDevices:BATTERY_SPRING_KEYSTONE5222 -> HyTechDevices:BATTERY_SPRING
Changed lines of the file:
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@@
 <layer number="154" name="FabDoc2" color="7" fill="1" visible="yes" active="yes"/>
 <layer number="155" name="FabDoc3" color="7" fill="1" visible="yes" active="yes"/>
-<layer number="156" name="HVSpacing" color="12" fill="1" visible="no" active="yes"/>
 <layer number="191" name="mNets" color="7" fill="1" visible="yes" active="yes"/>
 <layer number="192" name="mBusses" color="7" fill="1" visible="yes" active="yes"/>
@@
 </modules>
 <parts>
-<part name="CELL9" library="HyTechDevices" deviceset="BATTERY_SPRING" device="_KEYSTONE5222" value="BATTERY_SPRING_KEYSTONE5222"/>
-<part name="CELL8" library="HyTechDevices" deviceset="BATTERY_SPRING" device="_KEYSTONE5222" value="BATTERY_SPRING_KEYSTONE5222"/>
-<part name="CELL7" library="HyTechDevices" deviceset="BATTERY_SPRING" device="_KEYSTONE5222" value="BATTERY_SPRING_KEYSTONE5222"/>
-<part name="CELL6" library="HyTechDevices" deviceset="BATTERY_SPRING" device="_KEYSTONE5222" value="BATTERY_SPRING_KEYSTONE5222"/>
-<part name="CELL4" library="HyTechDevices" deviceset="BATTERY_SPRING" device="_KEYSTONE5222" value="BATTERY_SPRING_KEYSTONE5222"/>
-<part name="CELL5" library="HyTechDevices" deviceset="BATTERY_SPRING" device="_KEYSTONE5222" value="BATTERY_SPRING_KEYSTONE5222"/>
-<part name="CELL3" library="HyTechDevices" deviceset="BATTERY_SPRING" device="_KEYSTONE5222" value="BATTERY_SPRING_KEYSTONE5222"/>
-<part name="CELL2" library="HyTechDevices" deviceset="BATTERY_SPRING" device="_KEYSTONE5222" value="BATTERY_SPRING_KEYSTONE5222"/>
-<part name="CELL1" library="HyTechDevices" deviceset="BATTERY_SPRING" device="_KEYSTONE5222" value="BATTERY_SPRING_KEYSTONE5222"/>
-<part name="CELL0" library="HyTechDevices" deviceset="BATTERY_SPRING" device="_KEYSTONE5222" value="BATTERY_SPRING_KEYSTONE5222"/>
-<part name="CELL18" library="HyTechDevices" deviceset="BATTERY_SPRING" device="_KEYSTONE5222" value="BATTERY_SPRING_KEYSTONE5222"/>
-<part name="CELL17" library="HyTechDevices" deviceset="BATTERY_SPRING" device="_KEYSTONE5222" value="BATTERY_SPRING_KEYSTONE5222"/>
-<part name="CELL16" library="HyTechDevices" deviceset="BATTERY_SPRING" device="_KEYSTONE5222" value="BATTERY_SPRING_KEYSTONE5222"/>
-<part name="CELL15" library="HyTechDevices" deviceset="BATTERY_SPRING" device="_KEYSTONE5222" value="BATTERY_SPRING_KEYSTONE5222"/>
-<part name="CELL13" library="HyTechDevices" deviceset="BATTERY_SPRING" device="_KEYSTONE5222" value="BATTERY_SPRING_KEYSTONE5222"/>
-<part name="CELL14" library="HyTechDevices" deviceset="BATTERY_SPRING" device="_KEYSTONE5222" value="BATTERY_SPRING_KEYSTONE5222"/>
-<part name="CELL12" library="HyTechDevices" deviceset="BATTERY_SPRING" device="_KEYSTONE5222" value="BATTERY_SPRING_KEYSTONE5222"/>
-<part name="CELL11" library="HyTechDevices" deviceset="BATTERY_SPRING" device="_KEYSTONE5222" value="BATTERY_SPRING_KEYSTONE5222"/>
-<part name="CELL10" library="HyTechDevices" deviceset="BATTERY_SPRING" device="_KEYSTONE5222" value="BATTERY_SPRING_KEYSTONE5222"/>
+<part name="CELL9" library="HyTechDevices" deviceset="BATTERY_SPRING" device="" value="BATTERY_SPRING"/>
+<part name="CELL8" library="HyTechDevices" deviceset="BATTERY_SPRING" device="" value="BATTERY_SPRING"/>
+<part name="CELL7" library="HyTechDevices" deviceset="BATTERY_SPRING" device="" value="BATTERY_SPRING"/>
+<part name="CELL6" library="HyTechDevices" deviceset="BATTERY_SPRING" device="" value="BATTERY_SPRING"/>
+<part name="CELL4" library="HyTechDevices" deviceset="BATTERY_SPRING" device="" value="BATTERY_SPRING"/>
+<part name="CELL5" library="HyTechDevices" deviceset="BATTERY_SPRING" device="" value="BATTERY_SPRING"/>
+<part name="CELL3" library="HyTechDevices" deviceset="BATTERY_SPRING" device="" value="BATTERY_SPRING"/>
+<part name="CELL2" library="HyTechDevices" deviceset="BATTERY_SPRING" device="" value="BATTERY_SPRING"/>
+<part name="CELL1" library="HyTechDevices" deviceset="BATTERY_SPRING" device="" value="BATTERY_SPRING"/>
+<part name="CELL0" library="HyTechDevices" deviceset="BATTERY_SPRING" device="" value="BATTERY_SPRING"/>
+<part name="CELL18" library="HyTechDevices" deviceset="BATTERY_SPRING" device="" value="BATTERY_SPRING"/>
+<part name="CELL17" library="HyTechDevices" deviceset="BATTERY_SPRING" device="" value="BATTERY_SPRING"/>
+<part name="CELL16" library="HyTechDevices" deviceset="BATTERY_SPRING" device="" value="BATTERY_SPRING"/>
+<part name="CELL15" library="HyTechDevices" deviceset="BATTERY_SPRING" device="" value="BATTERY_SPRING"/>
+<part name="CELL13" library="HyTechDevices" deviceset="BATTERY_SPRING" device="" value="BATTERY_SPRING"/>
+<part name="CELL14" library="HyTechDevices" deviceset="BATTERY_SPRING" device="" value="BATTERY_SPRING"/>
+<part name="CELL12" library="HyTechDevices" deviceset="BATTERY_SPRING" device="" value="BATTERY_SPRING"/>
+<part name="CELL11" library="HyTechDevices" deviceset="BATTERY_SPRING" device="" value="BATTERY_SPRING"/>
+<part name="CELL10" library="HyTechDevices" deviceset="BATTERY_SPRING" device="" value="BATTERY_SPRING"/>
 <part name="A_LOWER_OUTPUT" library="HyTechDevices" deviceset="CONNECTOR-14" device=""/>
 <part name="A_LOWER_INPUT" library="HyTechDevices" deviceset="CONNECTOR-14" device=""/>
