File: EAGLE Board Designs/BMS/BMS Enerdel Adapter/BMS Enerdel Adapter rev5.brd (EAGLE design)
At the start: 108 x 331.4 mm, 27 parts

Commit message: Changed the mounting holes to the M4 mounting hole device from the HyTech Library and verified the board
Parts:
- added U$1, U$10, U$11, U$12, U$13, U$2, U$3, U$4, U$5, U$6, U$7, U$8, U$9: (no value), HyTechDevices:M4_MOUNTING
Routing:
- net A9-B15: track 403.2 -> 404.5 mm
Changed lines of the file:
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@@
 <wire x1="0" y1="280.384" x2="0" y2="223.93138125" width="0" layer="20"/>
 <wire x1="0" y1="223.93138125" x2="9" y2="223.93138125" width="0" layer="20"/>
-<hole x="5" y="234.284" drill="4.4958"/>
-<hole x="5" y="178.936" drill="4.4958"/>
-<hole x="5" y="148.986" drill="4.4958"/>
-<hole x="5" y="98.986" drill="4.4958"/>
-<hole x="5" y="69.046" drill="4.4958"/>
-<hole x="5" y="11.666" drill="4.4958"/>
-<hole x="101.65" y="38.114" drill="4.4958"/>
-<hole x="101.65" y="88.986" drill="4.4958"/>
-<hole x="103.65" y="158.986" drill="4.4958"/>
-<hole x="103.65" y="201.994" drill="4.4958"/>
 <wire x1="2" y1="-1.524" x2="93.3" y2="-1.524" width="1.27" layer="51"/>
 <text x="99.618" y="64.008" size="2.286" layer="51" font="vector" rot="R90" align="center">DANGER HIGH VOLTAGE</text>
@@
 <dimension x1="108" y1="28.702" x2="108" y2="212.82" x3="114.808" y3="120.761" textsize="2.54" layer="47"/>
 <text x="48.006" y="249.682" size="2.54" layer="52" font="vector" rot="MR180" align="center">DANGER HIGH VOLTAGE</text>
-<hole x="53.848" y="170.688" drill="4.4958"/>
-<hole x="53.848" y="121.412" drill="4.4958"/>
-<hole x="53.848" y="72.136" drill="4.4958"/>
 </plain>
 <attributes>
@@
 <element name="B_UPPER_OUTPUT1" library="HyTechDevices" package="NANO-FIT_VERTICAL-14" value="CONNECTOR-14NANO-FIT_VERTICAL-14" x="61.468" y="269.494" smashed="yes" rot="R90"/>
 <element name="B_UPPER_INPUT1" library="HyTechDevices" package="NANO-FIT_VERTICAL-14" value="CONNECTOR-14NANO-FIT_VERTICAL-14" x="86.868" y="269.494" smashed="yes" rot="R90"/>
+<element name="U$1" library="HyTechDevices" package="M4_MOUNTING" value="" x="5" y="11.666" smashed="yes"/>
+<element name="U$2" library="HyTechDevices" package="M4_MOUNTING" value="" x="5" y="69.046" smashed="yes"/>
+<element name="U$3" library="HyTechDevices" package="M4_MOUNTING" value="" x="5" y="98.986" smashed="yes"/>
+<element name="U$4" library="HyTechDevices" package="M4_MOUNTING" value="" x="5" y="148.986" smashed="yes"/>
+<element name="U$5" library="HyTechDevices" package="M4_MOUNTING" value="" x="5" y="178.936" smashed="yes"/>
+<element name="U$6" library="HyTechDevices" package="M4_MOUNTING" value="" x="5" y="234.284" smashed="yes"/>
+<element name="U$7" library="HyTechDevices" package="M4_MOUNTING" value="" x="103.65" y="201.994" smashed="yes"/>
+<element name="U$8" library="HyTechDevices" package="M4_MOUNTING" value="" x="103.65" y="158.986" smashed="yes"/>
+<element name="U$9" library="HyTechDevices" package="M4_MOUNTING" value="" x="101.65" y="88.986" smashed="yes"/>
+<element name="U$10" library="HyTechDevices" package="M4_MOUNTING" value="" x="101.65" y="38.114" smashed="yes"/>
+<element name="U$11" library="HyTechDevices" package="M4_MOUNTING" value="" x="53.848" y="72.136" smashed="yes"/>
+<element name="U$12" library="HyTechDevices" package="M4_MOUNTING" value="" x="53.848" y="121.412" smashed="yes"/>
+<element name="U$13" library="HyTechDevices" package="M4_MOUNTING" value="" x="53.848" y="170.688" smashed="yes"/>
 </elements>
 <signals>
@@
 <wire x1="37.61" y1="-39.388" x2="37.592" y2="-39.37" width="0.4064" layer="1"/>
 <wire x1="37.592" y1="-39.37" x2="35.56" y2="-41.402" width="0.4064" layer="1"/>
-<wire x1="39.326" y1="-39.388" x2="42.146" y2="-39.388" width="0.4064" layer="1"/>
-<wire x1="42.146" y1="-39.388" x2="50.038" y2="-31.496" width="0.4064" layer="1"/>
+<wire x1="39.326" y1="-39.388" x2="42.654" y2="-39.388" width="0.4064" layer="1"/>
+<wire x1="42.654" y1="-39.388" x2="49.276" y2="-32.766" width="0.4064" layer="1"/>
 <wire x1="89.662" y1="259.08" x2="87.884" y2="257.302" width="0.4064" layer="1"/>
 <wire x1="87.884" y1="257.302" x2="87.376" y2="256.794" width="0.4064" layer="1"/>
@@
 <via x="84.836" y="256.794" extent="1-16" drill="0.381"/>
 <wire x1="84.836" y1="256.794" x2="77.724" y2="256.794" width="0.4064" layer="1"/>
-<wire x1="50.038" y1="100.584" x2="50.038" y2="-31.496" width="0.4064" layer="1"/>
+<wire x1="49.276" y1="101.6" x2="49.276" y2="-32.766" width="0.4064" layer="1"/>
 <wire x1="88.392" y1="119.222" x2="88.392" y2="249.682" width="0.4064" layer="1"/>
 <via x="88.392" y="249.682" extent="1-16" drill="0.381"/>
@@
 <wire x1="73.914" y1="107.95" x2="77.12" y2="107.95" width="0.4064" layer="1"/>
 <wire x1="77.12" y1="107.95" x2="88.392" y2="119.222" width="0.4064" layer="1"/>
-<wire x1="73.914" y1="107.95" x2="57.404" y2="107.95" width="0.4064" layer="1"/>
-<wire x1="57.404" y1="107.95" x2="50.038" y2="100.584" width="0.4064" layer="1"/>
+<wire x1="73.914" y1="107.95" x2="55.626" y2="107.95" width="0.4064" layer="1"/>
+<wire x1="55.626" y1="107.95" x2="49.276" y2="101.6" width="0.4064" layer="1"/>
 </signal>
 <signal name="A10-B16">

Commit message: Adjusted schematic/board
Routing:
- net A7-B13: track 419.6 -> 417.7 mm
- net A1-B7: track 119.1 -> 118.3 mm
- net A12-B18: track 413.6 -> 413.0 mm
Other:
- board size 108 x 331.4 mm -> 108 x 333.9 mm
- board text added: "BMS Enerdel Adapter 2020 rev5"
- board text removed: "BMS Enerdel Adapter 2019 rev4"
- board text removed: "DO NOT MIX A & B"
