File: EAGLE Board Designs/BMS/BMS Enerdel Adapter/BMS Enerdel Adapter rev5.sch (EAGLE design)
At the start: 27 parts

Commit message: Made file changes so that the files were correctly named
Parts:
- CELL0, CELL1, CELL10, CELL11, CELL12, CELL13, CELL14, CELL15, CELL16, CELL17, CELL18, CELL2, CELL3, CELL4, CELL5, CELL6, CELL7, CELL8, CELL9: value BATTERY_SPRING -> BATTERY_SPRING_KEYSTONE5222; device HyTechDevices:BATTERY_SPRING -> HyTechDevices:BATTERY_SPRING_KEYSTONE5222
Changed lines of the file:
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@@
 <layer number="154" name="FabDoc2" color="7" fill="1" visible="yes" active="yes"/>
 <layer number="155" name="FabDoc3" color="7" fill="1" visible="yes" active="yes"/>
+<layer number="156" name="HVSpacing" color="12" fill="1" visible="no" active="yes"/>
 <layer number="191" name="mNets" color="7" fill="1" visible="yes" active="yes"/>
 <layer number="192" name="mBusses" color="7" fill="1" visible="yes" active="yes"/>
@@
 </modules>
 <parts>
-<part name="CELL9" library="HyTechDevices" deviceset="BATTERY_SPRING" device="" value="BATTERY_SPRING"/>
-<part name="CELL8" library="HyTechDevices" deviceset="BATTERY_SPRING" device="" value="BATTERY_SPRING"/>
-<part name="CELL7" library="HyTechDevices" deviceset="BATTERY_SPRING" device="" value="BATTERY_SPRING"/>
-<part name="CELL6" library="HyTechDevices" deviceset="BATTERY_SPRING" device="" value="BATTERY_SPRING"/>
-<part name="CELL4" library="HyTechDevices" deviceset="BATTERY_SPRING" device="" value="BATTERY_SPRING"/>
-<part name="CELL5" library="HyTechDevices" deviceset="BATTERY_SPRING" device="" value="BATTERY_SPRING"/>
-<part name="CELL3" library="HyTechDevices" deviceset="BATTERY_SPRING" device="" value="BATTERY_SPRING"/>
-<part name="CELL2" library="HyTechDevices" deviceset="BATTERY_SPRING" device="" value="BATTERY_SPRING"/>
-<part name="CELL1" library="HyTechDevices" deviceset="BATTERY_SPRING" device="" value="BATTERY_SPRING"/>
-<part name="CELL0" library="HyTechDevices" deviceset="BATTERY_SPRING" device="" value="BATTERY_SPRING"/>
-<part name="CELL18" library="HyTechDevices" deviceset="BATTERY_SPRING" device="" value="BATTERY_SPRING"/>
-<part name="CELL17" library="HyTechDevices" deviceset="BATTERY_SPRING" device="" value="BATTERY_SPRING"/>
-<part name="CELL16" library="HyTechDevices" deviceset="BATTERY_SPRING" device="" value="BATTERY_SPRING"/>
-<part name="CELL15" library="HyTechDevices" deviceset="BATTERY_SPRING" device="" value="BATTERY_SPRING"/>
-<part name="CELL13" library="HyTechDevices" deviceset="BATTERY_SPRING" device="" value="BATTERY_SPRING"/>
-<part name="CELL14" library="HyTechDevices" deviceset="BATTERY_SPRING" device="" value="BATTERY_SPRING"/>
-<part name="CELL12" library="HyTechDevices" deviceset="BATTERY_SPRING" device="" value="BATTERY_SPRING"/>
-<part name="CELL11" library="HyTechDevices" deviceset="BATTERY_SPRING" device="" value="BATTERY_SPRING"/>
-<part name="CELL10" library="HyTechDevices" deviceset="BATTERY_SPRING" device="" value="BATTERY_SPRING"/>
+<part name="CELL9" library="HyTechDevices" deviceset="BATTERY_SPRING" device="_KEYSTONE5222" value="BATTERY_SPRING_KEYSTONE5222"/>
+<part name="CELL8" library="HyTechDevices" deviceset="BATTERY_SPRING" device="_KEYSTONE5222" value="BATTERY_SPRING_KEYSTONE5222"/>
+<part name="CELL7" library="HyTechDevices" deviceset="BATTERY_SPRING" device="_KEYSTONE5222" value="BATTERY_SPRING_KEYSTONE5222"/>
+<part name="CELL6" library="HyTechDevices" deviceset="BATTERY_SPRING" device="_KEYSTONE5222" value="BATTERY_SPRING_KEYSTONE5222"/>
+<part name="CELL4" library="HyTechDevices" deviceset="BATTERY_SPRING" device="_KEYSTONE5222" value="BATTERY_SPRING_KEYSTONE5222"/>
+<part name="CELL5" library="HyTechDevices" deviceset="BATTERY_SPRING" device="_KEYSTONE5222" value="BATTERY_SPRING_KEYSTONE5222"/>
+<part name="CELL3" library="HyTechDevices" deviceset="BATTERY_SPRING" device="_KEYSTONE5222" value="BATTERY_SPRING_KEYSTONE5222"/>
+<part name="CELL2" library="HyTechDevices" deviceset="BATTERY_SPRING" device="_KEYSTONE5222" value="BATTERY_SPRING_KEYSTONE5222"/>
+<part name="CELL1" library="HyTechDevices" deviceset="BATTERY_SPRING" device="_KEYSTONE5222" value="BATTERY_SPRING_KEYSTONE5222"/>
+<part name="CELL0" library="HyTechDevices" deviceset="BATTERY_SPRING" device="_KEYSTONE5222" value="BATTERY_SPRING_KEYSTONE5222"/>
+<part name="CELL18" library="HyTechDevices" deviceset="BATTERY_SPRING" device="_KEYSTONE5222" value="BATTERY_SPRING_KEYSTONE5222"/>
+<part name="CELL17" library="HyTechDevices" deviceset="BATTERY_SPRING" device="_KEYSTONE5222" value="BATTERY_SPRING_KEYSTONE5222"/>
+<part name="CELL16" library="HyTechDevices" deviceset="BATTERY_SPRING" device="_KEYSTONE5222" value="BATTERY_SPRING_KEYSTONE5222"/>
+<part name="CELL15" library="HyTechDevices" deviceset="BATTERY_SPRING" device="_KEYSTONE5222" value="BATTERY_SPRING_KEYSTONE5222"/>
+<part name="CELL13" library="HyTechDevices" deviceset="BATTERY_SPRING" device="_KEYSTONE5222" value="BATTERY_SPRING_KEYSTONE5222"/>
+<part name="CELL14" library="HyTechDevices" deviceset="BATTERY_SPRING" device="_KEYSTONE5222" value="BATTERY_SPRING_KEYSTONE5222"/>
+<part name="CELL12" library="HyTechDevices" deviceset="BATTERY_SPRING" device="_KEYSTONE5222" value="BATTERY_SPRING_KEYSTONE5222"/>
+<part name="CELL11" library="HyTechDevices" deviceset="BATTERY_SPRING" device="_KEYSTONE5222" value="BATTERY_SPRING_KEYSTONE5222"/>
+<part name="CELL10" library="HyTechDevices" deviceset="BATTERY_SPRING" device="_KEYSTONE5222" value="BATTERY_SPRING_KEYSTONE5222"/>
 <part name="A_LOWER_OUTPUT" library="HyTechDevices" deviceset="CONNECTOR-14" device=""/>
 <part name="A_LOWER_INPUT" library="HyTechDevices" deviceset="CONNECTOR-14" device=""/>

Commit message: Adjusted schematic/board
Other:
- note removed: "Cell Input"
- note removed: "Gate Drive"
- note removed: "See LTC6804 DATASHEET pg.61"
Changed lines of the file:
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@@
 </class>
 </classes>
-<modules>
-<module name="DRAIN+FILTER" prefix="" dx="20.32" dy="15.24">
-<ports>
-<port name="CELL+" side="left" coord="5.08" direction="in"/>
-<port name="CELL-" side="left" coord="-5.08" direction="out"/>
-<port name="S(N)" side="right" coord="-5.08" direction="in"/>
-<port name="C(N)" side="right" coord="5.08" direction="out"/>
-<port name="V-" side="right" coord="0" direction="pwr"/>
-</ports>
-<variantdefs>
-</variantdefs>
-<parts>
-<part name="GATE" library="HyTechDevices" deviceset="RESISTOR" device="0805-RES" value="3.3kΩ"/>
-<part name="DISCHARGE" library="HyTechDevices" deviceset="RESISTOR" device="PWR163" value="5Ω"/>
-<part name="PFET" library="HyTechDevices" deviceset="P-CHANNEL_MOSFET_DMP3099L-7" device=""/>
-<part name="R" library="HyTechDevices" deviceset="RESISTOR" device="0805-RES" value="100Ω"/>
-<part name="C" library="HyTechDevices" deviceset="CAP" device="0805" value="10nF"/>
-<part name="SUPPLY1" library="supply2" deviceset="V-" device=""/>
-<part name="LED1" library="HyTechDevices" deviceset="LED" device="-0805" value="RED"/>
-<part name="R1" library="HyTechDevices" deviceset="RESISTOR" device="0805-RES" value="150"/>
-</parts>
-<sheets>
-<sheet>
-<plain>
-<text x="88.9" y="25.4" size="1.778" layer="97">Gate Drive</text>
-<text x="2.54" y="60.96" size="5.08" layer="97">See LTC6804 DATASHEET pg.61</text>
-<text x="88.9" y="43.18" size="1.778" layer="97">Cell Input</text>
-</plain>
-<instances>
-<instance part="GATE" gate="G$1" x="55.88" y="25.4" smashed="yes">
-<attribute name="NAME" x="52.07" y="26.8986" size="1.778" layer="95"/>
-<attribute name="VALUE" x="52.07" y="22.098" size="1.778" layer="96"/>
-</instance>
-<instance part="DISCHARGE" gate="G$1" x="35.56" y="12.7" smashed="yes" rot="R270">
-<attribute name="NAME" x="37.0586" y="16.51" size="1.778" layer="95" rot="R270"/>
-<attribute name="VALUE" x="32.258" y="16.51" size="1.778" layer="96" rot="R270"/>
-</instance>
-<instance part="PFET" gate="G$1" x="40.64" y="22.86" smashed="yes" rot="R180">
-<attribute name="NAME" x="36.83" y="27.94" size="1.778" layer="95"/>
-</instance>
-<instance part="R" gate="G$1" x="55.88" y="43.18" smashed="yes">
-<attribute name="NAME" x="52.07" y="44.6786" size="1.778" layer="95"/>
-<attribute name="VALUE" x="52.07" y="39.878" size="1.778" layer="96"/>
-</instance>
-<instance part="C" gate="G$1" x="68.58" y="35.56" smashed="yes">
-<attribute name="NAME" x="70.104" y="38.481" size="1.778" layer="95"/>
-<attribute name="VALUE" x="70.104" y="33.401" size="1.778" layer="96"/>
-</instance>
-<instance part="SUPPLY1" gate="1" x="68.58" y="27.94" smashed="yes">
-<attribute name="VALUE" x="67.31" y="25.4" size="1.778" layer="96"/>
-</instance>
-<instance part="LED1" gate="LED" x="22.86" y="20.32" smashed="yes" rot="R270">
-<attribute name="NAME" x="18.288" y="16.764" size="1.778" layer="95"/>
-<attribute name="VALUE" x="18.288" y="14.605" size="1.778" layer="96"/>
-</instance>
-<instance part="R1" gate="G$1" x="10.16" y="20.32" smashed="yes">
-<attribute name="NAME" x="6.35" y="21.8186" size="1.778" layer="95"/>
-<attribute name="VALUE" x="6.35" y="17.018" size="1.778" layer="96"/>
-</instance>
-</instances>
-<busses>
-</busses>
-<nets>
-<net name="CELL+" class="0">
-<segment>
-<wire x1="35.56" y1="43.18" x2="35.56" y2="25.4" width="0.1524" layer="91"/>
-<wire x1="35.56" y1="43.18" x2="27.94" y2="43.18" width="0.1524" layer="91"/>
-<pinref part="PFET" gate="G$1" pin="S"/>
-<label x="27.94" y="43.18" size="1.778" layer="95" rot="R180" xref="yes"/>
-<pinref part="R" gate="G$1" pin="1"/>
-<wire x1="50.8" y1="43.18" x2="35.56" y2="43.18" width="0.1524" layer="91"/>
-<junction x="35.56" y="43.18"/>
-</segment>
-</net>
-<net name="GATE" class="0">
-<segment>
-<pinref part="GATE" gate="G$1" pin="1"/>
-<wire x1="45.72" y1="25.4" x2="50.8" y2="25.4" width="0.1524" layer="91"/>
-<pinref part="PFET" gate="G$1" pin="G"/>
-</segment>
-</net>
-<net name="S(N)" class="0">
-<segment>
-<pinref part="GATE" gate="G$1" pin="2"/>
-<wire x1="60.96" y1="25.4" x2="78.74" y2="25.4" width="0.1524" layer="91"/>
-<label x="78.74" y="25.4" size="1.778" layer="95" xref="yes"/>
-</segment>
-</net>
-<net name="CELL-" class="0">
-<segment>
-<wire x1="35.56" y1="5.08" x2="27.94" y2="5.08" width="0.1524" layer="91"/>
-<label x="27.94" y="5.08" size="1.778" layer="95" rot="R180" xref="yes"/>
-<pinref part="DISCHARGE" gate="G$1" pin="2"/>
-<wire x1="35.56" y1="7.62" x2="35.56" y2="5.08" width="0.1524" layer="91"/>
-</segment>
-<segment>
-<pinref part="R1" gate="G$1" pin="1"/>
-<wire x1="5.08" y1="20.32" x2="2.54" y2="20.32" width="0.1524" layer="91"/>
-<label x="2.54" y="20.32" size="1.778" layer="95" rot="R180" xref="yes"/>
-</segment>
-</net>
-<net name="C(N)" class="0">
-<segment>
-<pinref part="R" gate="G$1" pin="2"/>
-<pinref part="C" gate="G$1" pin="1"/>
-<wire x1="60.96" y1="43.18" x2="68.58" y2="43.18" width="0.1524" layer="91"/>
-<wire x1="68.58" y1="43.18" x2="68.58" y2="40.64" width="0.1524" layer="91"/>
-<wire x1="68.58" y1="43.18" x2="78.74" y2="43.18" width="0.1524" layer="91"/>
-<junction x="68.58" y="43.18"/>
-<label x="78.74" y="43.18" size="1.778" layer="95" xref="yes"/>
-</segment>
-</net>
-<net name="V-" class="0">
-<segment>
-<pinref part="C" gate="G$1" pin="2"/>
-<wire x1="68.58" y1="33.02" x2="68.58" y2="30.48" width="0.1524" layer="91"/>
-<pinref part="SUPPLY1" gate="1" pin="V-"/>
-</segment>
-</net>
-<net name="N$1" class="0">
-<segment>
-<pinref part="PFET" gate="G$1" pin="D"/>
-<pinref part="DISCHARGE" gate="G$1" pin="1"/>
-<wire x1="35.56" y1="20.32" x2="35.56" y2="17.78" width="0.1524" layer="91"/>
-<pinref part="LED1" gate="LED" pin="A"/>
-<wire x1="35.56" y1="20.32" x2="25.4" y2="20.32" width="0.1524" layer="91"/>
-<junction x="35.56" y="20.32"/>
-</segment>
-</net>
-<net name="N$2" class="0">
-<segment>
-<pinref part="LED1" gate="LED" pin="C"/>
-<pinref part="R1" gate="G$1" pin="2"/>
-<wire x1="15.24" y1="20.32" x2="17.78" y2="20.32" width="0.1524" layer="91"/>
-</segment>
-</net>
-</nets>
-</sheet>
-</sheets>
-</module>
-<module name="THERM_FILTER" prefix="" dx="22.86" dy="15.24">
-<ports>
-<port name="VREF" side="left" coord="5.08" direction="pwr"/>
-<port name="GPIO" side="left" coord="-5.08" direction="out"/>
-<port name="THERM" side="right" coord="-5.08" direction="nc"/>
-<port name="V-" side="right" coord="5.08" direction="pwr"/>
-</ports>
-<variantdefs>
-</variantdefs>
-<parts>
-<part name="R1" library="HyTechDevices" deviceset="RESISTOR" device="0805-RES" value="10kΩ"/>
-<part name="R" library="HyTechDevices" deviceset="RESISTOR" device="0805-RES" value="100Ω"/>
-<part name="C" library="HyTechDevices" deviceset="CAP" device="0805" value="10nF"/>
-<part name="SUPPLY27" library="supply2" deviceset="V-" device=""/>
-</parts>
-<sheets>
-<sheet>
-<plain>
-</plain>
-<instances>
-<instance part="R1" gate="G$1" x="10.16" y="10.16" smashed="yes" rot="R270">
-<attribute name="NAME" x="11.6586" y="13.97" size="1.778" layer="95" rot="R270"/>
-<attribute name="VALUE" x="6.858" y="13.97" size="1.778" layer="96" rot="R270"/>
-</instance>
-<instance part="R" gate="G$1" x="0" y="0" smashed="yes">
-<attribute name="NAME" x="-3.81" y="1.4986" size="1.778" layer="95"/>
-<attribute name="VALUE" x="-3.81" y="-3.302" size="1.778" layer="96"/>
-</instance>
-<instance part="C" gate="G$1" x="-10.16" y="-7.62" smashed="yes">
-<attribute name="NAME" x="-8.636" y="-4.699" size="1.778" layer="95"/>
-<attribute name="VALUE" x="-8.636" y="-9.779" size="1.778" layer="96"/>
-</instance>
-<instance part="SUPPLY27" gate="1" x="-10.16" y="-15.24" smashed="yes">
-<attribute name="VALUE" x="-11.43" y="-17.78" size="1.778" layer="96"/>
-</instance>
-</instances>
-<busses>
-</busses>
-<nets>
-<net name="THERM" class="0">
-<segment>
-<pinref part="R1" gate="G$1" pin="2"/>
-<wire x1="10.16" y1="-7.62" x2="10.16" y2="0" width="0.1524" layer="91"/>
-<pinref part="R" gate="G$1" pin="2"/>
-<wire x1="10.16" y1="0" x2="10.16" y2="5.08" width="0.1524" layer="91"/>
-<wire x1="5.08" y1="0" x2="10.16" y2="0" width="0.1524" layer="91"/>
-<junction x="10.16" y="0"/>
-<label x="10.16" y="-7.62" size="1.778" layer="95" rot="R270" xref="yes"/>
-</segment>
-</net>
-<net name="GPIO" class="0">
-<segment>
-<pinref part="R" gate="G$1" pin="1"/>
-<pinref part="C" gate="G$1" pin="1"/>
-<wire x1="-10.16" y1="-2.54" x2="-10.16" y2="0" width="0.1524" layer="91"/>
-<wire x1="-10.16" y1="0" x2="-5.08" y2="0" width="0.1524" layer="91"/>
-<wire x1="-10.16" y1="0" x2="-17.78" y2="0" width="0.1524" layer="91"/>
-<junction x="-10.16" y="0"/>
-<label x="-17.78" y="0" size="1.778" layer="95" rot="R180" xref="yes"/>
-</segment>
-</net>
-<net name="VREF" class="0">
-<segment>
-<pinref part="R1" gate="G$1" pin="1"/>
-<wire x1="10.16" y1="15.24" x2="10.16" y2="17.78" width="0.1524" layer="91"/>
-<label x="10.16" y="17.78" size="1.778" layer="95" rot="R90" xref="yes"/>
-</segment>
-</net>
-<net name="V-" class="0">
-<segment>
-<pinref part="SUPPLY27" gate="1" pin="V-"/>
-<pinref part="C" gate="G$1" pin="2"/>
-<wire x1="-10.16" y1="-12.7" x2="-10.16" y2="-10.16" width="0.1524" layer="91"/>
-</segment>
-</net>
-</nets>
-</sheet>
-</sheets>
-</module>
-</modules>
 <parts>
 <part name="CELL9" library="HyTechDevices" deviceset="BATTERY_SPRING" device="_KEYSTONE5222" value="BATTERY_SPRING_KEYSTONE5222"/>

Commit message: Added frame to schematic and measures to board
Other:
- note added: "BMS Contacts"
- note added: "Cody Kaminsky"
- note added: "Enerdel Adapter for Testing BMS rev13 and BMS rev14 Boards"
Changed lines of the file:
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@@
 <part name="B_UPPER_OUTPUT1" library="HyTechDevices" deviceset="CONNECTOR-14" device="NANO-FIT_VERTICAL-14"/>
 <part name="B_UPPER_INPUT1" library="HyTechDevices" deviceset="CONNECTOR-14" device="NANO-FIT_VERTICAL-14"/>
+<part name="U$14" library="HyTechFrames" deviceset="FRAME_B" device=""/>
 </parts>
 <sheets>
 <sheet>
+<description>Enerdel Adapter for Testing BMS rev13 and BMS rev14 Boards</description>
 <plain>
-<wire x1="0" y1="157.48" x2="0" y2="0" width="1.27" layer="90"/>
-<wire x1="0" y1="0" x2="139.7" y2="0" width="1.27" layer="90"/>
-<wire x1="139.7" y1="0" x2="139.7" y2="157.48" width="1.27" layer="90"/>
-<wire x1="139.7" y1="157.48" x2="0" y2="157.48" width="1.27" layer="90"/>
-<wire x1="342.9" y1="157.48" x2="203.2" y2="157.48" width="1.27" layer="90"/>
-<wire x1="203.2" y1="157.48" x2="203.2" y2="0" width="1.27" layer="90"/>
-<wire x1="203.2" y1="0" x2="342.9" y2="0" width="1.27" layer="90"/>
-<wire x1="342.9" y1="0" x2="342.9" y2="157.48" width="1.27" layer="90"/>
-<text x="2.54" y="160.02" size="7.62" layer="90">A Mode</text>
-<text x="205.74" y="160.02" size="7.62" layer="90">B Mode</text>
-<text x="167.64" y="187.96" size="7.62" layer="90" align="center">Warning: only install Mode A or Mode B connectors
+<text x="58.42" y="152.4" size="7.62" layer="97">A Mode</text>
+<text x="261.62" y="152.4" size="7.62" layer="97">B Mode</text>
+<text x="167.64" y="187.96" size="7.62" layer="97" align="center">Warning: only install Mode A or Mode B connectors
 Do not use connectors from both modes</text>
+<text x="241.3" y="-30.48" size="2.54" layer="94">Cody Kaminsky</text>
+<text x="288.29" y="-43.18" size="2.54" layer="94">Enerdel Adapter for Testing BMS rev13 and BMS rev14 Boards</text>
+<text x="134.62" y="109.22" size="7.62" layer="97">BMS Contacts</text>
 </plain>
 <instances>
@@
 <attribute name="NAME" x="289.56" y="137.922" size="1.524" layer="95" rot="MR180"/>
 </instance>
+<instance part="U$14" gate="G$1" x="-40.64" y="-53.34" smashed="yes"/>
+<instance part="U$14" gate="G$2" x="222.25" y="-53.34" smashed="yes">
+<attribute name="LAST_DATE_TIME" x="298.45" y="-50.8" size="2.54" layer="94"/>
+<attribute name="DRAWING_NAME" x="317.5" y="-30.48" size="2.54" layer="94"/>
+<attribute name="SHEET" x="370.84" y="-50.8" size="2.54" layer="94"/>
+</instance>
 </instances>
