File: ESF Schematics/Shutdown Circuit.sch (EAGLE design)
At the start: 52 parts, among them J115F11A12VDCS6.9 RELAY

Commit message: updated ESF schematics
Other:
- note added: "Cable between GLV_BATTERY and FUSE2 is 14AWG. Shutdown Circuit after FUSE2 uses 18AWG cable and 22AWG after FUSE3. IMD_OK output uses 22AWG cable. DC-DC output uses 16 AWG cable. Thick green: 22AWG. Thick orange: aluminum busbars, 0.063875 inch^2"
- note removed: "Cable between GLV_BATTERY and FUSE2 is 14AWG. Shutdown Circuit after FUSE2 uses 18AWG cable and 22AWG after FUSE3. IMD_OK output uses 22AWG cable. DC-DC output uses 16 AWG cable. Thick green: 22AWG. Thick orange: aluminum busbars, 0.0625 inch^2"
Changed lines of the file:
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@@
 IMD_OK output uses 22AWG cable. DC-DC output uses 16 AWG cable.
 Thick green: 22AWG.
-Thick orange: aluminum busbars, 0.0625 inch^2</text>
+Thick orange: aluminum busbars, 0.063875 inch^2</text>
 <text x="129.54" y="22.86" size="2.54" layer="97">Shaan Dhawan</text>
 <text x="195.58" y="15.24" size="2.54" layer="97">HT05 safety circuitry schematic.</text>
