File: EAGLE Board Designs/BMS/BMS Segment/BMS Segment rev15 - Copy.brd (EAGLE design)
At the start: 108 x 240.3 mm, 239 parts, among them J0 CONNECTOR-1, J1 CONNECTOR-1, J10 CONNECTOR-1, J11 CONNECTOR-1, J12 CONNECTOR-1, J13 CONNECTOR-1, J14 CONNECTOR-1, J15 CONNECTOR-1, J16 CONNECTOR-1, J17 CONNECTOR-1, J18 CONNECTOR-1, J2 CONNECTOR-1, J3 CONNECTOR-1, J4 CONNECTOR-1, J5 CONNECTOR-1, J6 CONNECTOR-1, J7 CONNECTOR-1, J8 CONNECTOR-1, J9 CONNECTOR-1, T1 TRANSFORMERHM2102NLT, U1 LTC6813

Commit message: trying eagle hack
Parts:
- moved THERM9:C1 2315.7 mm to (-247.3, 1096.0)
- moved THERM8:C1 2301.4 mm to (-247.3, 1084.6)
- moved THERM7:C1 2289.9 mm to (-247.3, 1076.0)
- moved THERM6:C1 2268.0 mm to (-247.3, 1057.0)
- moved THERM5:C1 2254.8 mm to (-238.4, 1046.5)
- moved THERM4:C1 2232.7 mm to (-247.3, 1027.4)
- moved THERM3:C1 2219.5 mm to (-238.4, 1017.0)
- moved THERM2:C1 2197.4 mm to (-247.3, 997.9)
- moved CELL18:C1 2179.9 mm to (-172.4, 983.6)
- moved CELL17:C1 2151.9 mm to (-172.4, 958.5)
- moved C6 2136.2 mm to (-174.6, 992.2)
- moved CELL16:C1 2123.9 mm to (-172.4, 933.5)
- moved CELL15:C1 2095.9 mm to (-172.4, 908.4)
- moved CELL14:C1 2068.0 mm to (-172.4, 883.3)
- moved CELL13:C1 2040.0 mm to (-172.4, 858.2)
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Connections:
- removed net N$3: C8.1, T1.8
- new net N$17: C7.1, T1.8
- net N$5: now also C8.2; no longer C7.2
- net V-: now also C7.2, C8.1; no longer C7.1, C8.2
