File: EAGLE Board Designs/BMS/BMS Segment/BMS Segment rev15.brd (EAGLE design)
At the start: 108 x 240.3 mm, 239 parts, among them J0 CONNECTOR-1, J1 CONNECTOR-1, J10 CONNECTOR-1, J11 CONNECTOR-1, J12 CONNECTOR-1, J13 CONNECTOR-1, J14 CONNECTOR-1, J15 CONNECTOR-1, J16 CONNECTOR-1, J17 CONNECTOR-1, J18 CONNECTOR-1, J2 CONNECTOR-1, J3 CONNECTOR-1, J4 CONNECTOR-1, J5 CONNECTOR-1, J6 CONNECTOR-1, J7 CONNECTOR-1, J8 CONNECTOR-1, J9 CONNECTOR-1, T1 TRANSFORMERHM2102NLT, U1 LTC6813

Commit message: Resolved part cache error
Parts:
- removed Q3: (no value), HyTechDevices:SOT223
- added Q1: (no value), HyTechDevices:SOT223
Connections:
- net N$11: now also Q1.1; no longer Q3.1
- net N$12: now also Q1.3; no longer Q3.3
- net N$15: now also Q1.2, Q1.4; no longer Q3.2, Q3.4
Changed lines of the file:
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@@
 <element name="U$18" library="HyTechDevices" package="M4_MOUNTING" value="" x="53.848" y="72.136" smashed="yes"/>
 <element name="U$19" library="HyTechDevices" package="M4_MOUNTING" value="" x="53.848" y="121.412" smashed="yes"/>
-<element name="Q3" library="HyTechDevices" package="SOT223" value="" x="-25.0825" y="-18.415" smashed="yes">
-<attribute name="DKPN" value="NSV1C201MZ4T1GOSCT-ND" x="-25.0825" y="-18.415" size="1.778" layer="27" display="off"/>
-<attribute name="MANUFACTURER" value="ON Semiconductor" x="-25.0825" y="-18.415" size="1.778" layer="27" display="off"/>
-<attribute name="MOPN" value="863-NSV1C201MZ4T1G" x="-25.0825" y="-18.415" size="1.778" layer="27" display="off"/>
-<attribute name="MPN" value="NSV1C201MZ4" x="-25.0825" y="-18.415" size="1.778" layer="27" display="off"/>
-<attribute name="NAME" x="-25.0825" y="-13.97" size="0.8128" layer="25" font="vector" align="bottom-center"/>
-</element>
 <element name="R1" library="HyTechDevices" package="0603-RES" value="RESISTOR_0603_100" x="-26.67" y="-49.8475" smashed="yes">
 <attribute name="DKPN" value="311-100HRCT-ND" x="-26.67" y="-49.8475" size="1.778" layer="27" display="off"/>
@@
 <attribute name="VOLTAGE" value="100V" x="-293.37" y="-1219.2" size="1.778" layer="27" display="off"/>
 </element>
+<element name="Q1" library="HyTechDevices" package="SOT223" value="" x="-292.735" y="1110.9325" smashed="yes">
+<attribute name="DKPN" value="NSV1C201MZ4T1GOSCT-ND" x="-300.6725" y="-1215.7075" size="1.778" layer="27" display="off"/>
+<attribute name="MANUFACTURER" value="ON Semiconductor" x="-300.6725" y="-1215.7075" size="1.778" layer="27" display="off"/>
+<attribute name="MOPN" value="863-NSV1C201MZ4T1G" x="-300.6725" y="-1215.7075" size="1.778" layer="27" display="off"/>
+<attribute name="MPN" value="NSV1C201MZ4" x="-300.6725" y="-1215.7075" size="1.778" layer="27" display="off"/>
+<attribute name="NAME" x="-292.735" y="1115.3775" size="0.8128" layer="25" font="vector" align="bottom-center"/>
+</element>
 </elements>
 <signals>
 <signal name="N$11">
-<contactref element="Q3" pad="1"/>
 <contactref element="U1" pad="49"/>
-<wire x1="-27.3825" y1="-21.615" x2="-108.645" y2="-221.8975" width="0" layer="19" extent="1-1"/>
+<contactref element="Q1" pad="1"/>
+<wire x1="-295.035" y1="1107.7325" x2="-108.645" y2="-221.8975" width="0" layer="19" extent="1-1"/>
 </signal>
 <signal name="N$12">
-<contactref element="Q3" pad="3"/>
 <contactref element="U1" pad="52"/>
 <contactref element="U1" pad="48"/>
 <contactref element="U1" pad="55"/>
 <contactref element="C3" pad="1"/>
+<contactref element="Q1" pad="3"/>
 <wire x1="-110.145" y1="-221.8975" x2="-266.815" y2="-1122.045" width="0" layer="19" extent="1-1"/>
 <wire x1="-111.645" y1="-221.8975" x2="-110.145" y2="-221.8975" width="0" layer="19" extent="1-1"/>
 <wire x1="-106.645" y1="-223.8975" x2="-110.145" y2="-221.8975" width="0" layer="19" extent="1-1"/>
-<wire x1="-22.7825" y1="-21.615" x2="-110.145" y2="-221.8975" width="0" layer="19" extent="1-1"/>
+<wire x1="-290.435" y1="1107.7325" x2="-266.815" y2="-1122.045" width="0" layer="19" extent="1-1"/>
 </signal>
 <signal name="N$25">
@@
 </signal>
 <signal name="N$15">
-<contactref element="Q3" pad="4"/>
-<contactref element="Q3" pad="2"/>
 <contactref element="R1" pad="1"/>
 <contactref element="C4" pad="1"/>
+<contactref element="Q1" pad="4"/>
+<contactref element="Q1" pad="2"/>
 <wire x1="-27.52" y1="-49.8475" x2="-266.815" y2="-1124.9025" width="0" layer="19" extent="1-1"/>
-<wire x1="-25.0825" y1="-21.615" x2="-27.52" y2="-49.8475" width="0" layer="19" extent="1-1"/>
-<wire x1="-25.0825" y1="-15.215" x2="-25.0825" y2="-21.615" width="0" layer="19" extent="1-1"/>
+<wire x1="-292.735" y1="1114.1325" x2="-266.815" y2="-1124.9025" width="0" layer="19" extent="1-1"/>
+<wire x1="-292.735" y1="1107.7325" x2="-292.735" y2="1114.1325" width="0" layer="19" extent="1-1"/>
 </signal>
 <signal name="N$1">

Commit message: Basic work
Parts:
- moved J19 1270.1 mm to (103.2, 144.8), turned to 90 degrees
- moved J20 1240.5 mm to (102.9, 112.4), turned to 90 degrees
- moved C10 1011.0 mm to (-40.3, -153.7)
- moved C3 1011.0 mm to (-40.3, -136.5)
- moved C8 1011.0 mm to (-40.3, -145.1)
- moved CELL12:C1 1011.0 mm to (-48.6, -190.8)
- moved CELL15:C1 1011.0 mm to (-52.4, -199.4)
- moved CELL18:C1 1011.0 mm to (-56.2, -208.0)
- moved CELL1:D1 1011.0 mm to (69.5, -102.2)
- moved CELL1:R4 1011.0 mm to (52.7, -110.8)
- moved CELL6:C1 1011.0 mm to (-43.5, -173.7)
- moved CELL9:C1 1011.0 mm to (-45.4, -182.2)
- moved THERM1:R2 1011.0 mm to (-21.6, -128.0)
- moved THERM3:C1 1011.0 mm to (-60.0, -216.5)
- moved THERM6:C1 1011.0 mm to (-63.8, -225.1)
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Connections:
- net N$11 renamed DRIVE
- net N$12 renamed VREG
- net N$25 renamed VREF1
- net IMA: now also T1.12; no longer T1.9
- net IMB: now also T1.9; no longer T1.12
- net IPA: now also T1.10; no longer T1.7
- net IPB: now also T1.7; no longer T1.10
- net ISO_IMA: now also T1.1; no longer T1.4
- net ISO_IMB: now also T1.4; no longer T1.1
- net ISO_IPA: now also T1.3; no longer T1.6
- net ISO_IPB: now also T1.6; no longer T1.3
- net N$3: now also T1.11; no longer T1.8
- net N$4: now also T1.8; no longer T1.11

Commit message: Revert "Basic work"
This reverts commit 314f29d0700f840b339ecbc3c92328a4e326f93a.
Parts:
- moved J19 1270.1 mm to (-180.7, -1093.2), turned to 0 degrees
- moved J20 1240.5 mm to (-189.5, -1093.2), turned to 0 degrees
- moved C10 1011.0 mm to (-266.1, -1139.2)
- moved C3 1011.0 mm to (-266.1, -1122.0)
- moved C8 1011.0 mm to (-266.1, -1130.6)
- moved CELL12:C1 1011.0 mm to (-274.3, -1176.3)
- moved CELL15:C1 1011.0 mm to (-278.1, -1184.9)
- moved CELL18:C1 1011.0 mm to (-281.9, -1193.5)
- moved CELL1:D1 1011.0 mm to (-156.2, -1087.8)
- moved CELL1:R4 1011.0 mm to (-173.0, -1096.3)
- moved CELL6:C1 1011.0 mm to (-269.2, -1159.2)
- moved CELL9:C1 1011.0 mm to (-271.1, -1167.8)
- moved THERM1:R2 1011.0 mm to (-247.3, -1113.5)
- moved THERM3:C1 1011.0 mm to (-285.8, -1202.1)
- moved THERM6:C1 1011.0 mm to (-289.6, -1210.6)
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Connections:
- net DRIVE renamed N$11
- net VREF1 renamed N$25
- net VREG renamed N$12
- net IMA: now also T1.9; no longer T1.12
- net IMB: now also T1.12; no longer T1.9
- net IPA: now also T1.7; no longer T1.10
- net IPB: now also T1.10; no longer T1.7
- net ISO_IMA: now also T1.4; no longer T1.1
- net ISO_IMB: now also T1.1; no longer T1.4
- net ISO_IPA: now also T1.6; no longer T1.3
- net ISO_IPB: now also T1.3; no longer T1.6
- net N$3: now also T1.8; no longer T1.11
- net N$4: now also T1.11; no longer T1.8

Commit message: Reset board design
Parts:
- moved THERM9:C1 1448.6 mm to (-125.7, 219.7)
- moved THERM8:C1 1448.5 mm to (-102.9, 219.7)
- moved THERM7:C1 1434.4 mm to (-171.4, 215.9)
- moved THERM6:C1 1433.5 mm to (-148.6, 215.9)
- moved THERM5:C1 1432.9 mm to (-125.7, 215.9)
- moved THERM4:C1 1432.7 mm to (-102.9, 215.9)
- moved THERM3:C1 1416.5 mm to (-184.2, 210.8)
- moved THERM2:C1 1415.4 mm to (-161.3, 210.8)
- moved THERM1:C1 1414.6 mm to (-138.4, 210.8)
- moved C6 1365.5 mm to (-165.1, 219.7)
- moved C10 1361.6 mm to (-180.3, 219.7)
- moved C9 1359.0 mm to (-176.5, 219.7)
- moved C5 1357.2 mm to (-161.3, 219.7)
- moved C8 1353.6 mm to (-172.7, 219.7)
- moved C7 1351.0 mm to (-168.9, 219.7)
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Other:
- board text removed: "#"
- board text removed: "+"
- board text removed: "-"
- board text removed: "0"
- board text removed: "1"
- board text removed: "10"
- board text removed: "11"
- board text removed: "12"
- board text removed: "13"
- board text removed: "14"
- board text removed: "15"
- board text removed: "16"
- board text removed: "17"
- board text removed: "2"
- board text removed: "3"
- board text removed: "4"
- board text removed: "5"
- board text removed: "6"
- board text removed: "7"
- board text removed: "8"
- board text removed: "9"
- board text removed: "Cell 0"
- board text removed: "Cell 17"
- board text removed: "DANGER HIGH VOLTAGE"
- board text removed: "DRIVE_A"
- board text removed: "DRIVE_B"
- board text removed: "HyTech Racing 2020 BMS Segment rev14 Designed by Arvind Srinivasan, based on rev10 by Yvonne Yeh"
- board text removed: "TS"
- board text removed: "V-_A"
- board text removed: "V-_B"
- board text removed: "isoSPI"
- board text removed: "x1"
- board text removed: "x2"
- board text removed: "x4"
- board text removed: "x8"

Commit message: Minor BMS stuff
Parts:
- moved T1 135.6 mm to (-33.0, 121.9), turned to 90 degrees
- moved U1 106.4 mm to (-52.1, 121.9), turned to 270 degrees
- moved J0 2.54 mm to (-171.4, 203.2)
- moved J1 2.54 mm to (-175.3, 203.2)
- moved J2 2.54 mm to (-179.1, 203.2)
- moved J3 2.54 mm to (-182.9, 203.2)
- moved J4 2.54 mm to (-186.7, 203.2)
- moved J5 2.54 mm to (-190.5, 203.2)
- moved J6 2.54 mm to (-194.3, 203.2)
- moved J7 2.54 mm to (-198.1, 203.2)
- moved J8 2.54 mm to (-201.9, 203.2)
- moved J9 2.54 mm to (-205.7, 203.2)

Commit message: bms work
Parts:
- removed C10, C4, C9: (no value), HyTechDevices:0603-CAP
- removed R7: RESISTOR_0603_100, HyTechDevices:0603-RES
- removed R8, R9: RESISTOR_0603_1K, HyTechDevices:0603-RES
- added CELL0.C1, DRIVE.C1, SENSE18.C1: (no value), HyTechDevices:0603-CAP
- added CELL0.R1, DRIVE.R1, SENSE18.R1: RESISTOR_0603_100, HyTechDevices:0603-RES
- R1: value RESISTOR_0603_100 -> RESISTOR_0603_1K
- R2: value RESISTOR_0603_60.4 -> RESISTOR_0603_1K
- R3: value RESISTOR_0603_100 -> RESISTOR_0603_60.4
- moved R2 1138.2 mm to (-617.2, -834.4)
- moved R1 1136.1 mm to (-617.2, -830.6)
- moved C8 1133.0 mm to (-616.0, -823.0)
- moved C7 1131.0 mm to (-616.0, -819.1)
- moved C6 1129.0 mm to (-616.0, -815.3)
- moved C5 1127.0 mm to (-616.0, -811.5)
- moved C3 1108.8 mm to (-614.7, -788.7)
- moved C2 1106.9 mm to (-614.7, -784.9)
- moved R6 1106.8 mm to (-614.7, -807.7)
- moved C1 1105.0 mm to (-614.7, -781.0)
- moved R5 1104.7 mm to (-614.7, -803.9)
- moved R4 1102.6 mm to (-614.7, -800.1)
- moved R3 1100.5 mm to (-614.7, -796.3)
- moved J24 1044.5 mm to (-577.9, -759.5)
- moved J25 1044.5 mm to (-586.7, -759.5)
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Connections:
- net N$11 renamed DRIVE
- net N$12 renamed VREG
- net C0: now also CELL0.C1.1, CELL0.R1.2; no longer C10.1, R7.2
- net C18: no longer R1.2, R3.1
- net GPIO1: now also J27.1; no longer J28.1
- net GPIO1_PRE: now also J27.2; no longer J28.2
- net IMA: now also R3.1; no longer R6.1
- net IMB: now also R5.1; no longer R2.1
- net IPA: now also R4.2; no longer R5.2
- net IPB: now also R6.2; no longer R4.2
- net ISO_IMA: now also J25.2; no longer J19.2
- net ISO_IMB: now also J26.2; no longer J20.2
- net ISO_IPA: now also J25.1; no longer J19.1
- net ISO_IPB: now also J26.1; no longer J20.1
- net N$1: now also R1.2, R2.1; no longer R8.1, R9.2
- net N$15: now also DRIVE.C1.1, DRIVE.R1.2; no longer C4.1, R1.1
- net N$18: now also C8.2, R5.2, R6.1; no longer C9.2, R2.2, R4.1
- net N$2: now also R2.2; no longer R8.2
- net N$3: now also C5.1; no longer C8.1
- net N$4: now also C7.1; no longer C5.1
- net N$5: now also C6.2, R3.2, R4.1; no longer C7.2, R5.1, R6.2
- net SENSE17: now also J28.2; no longer J27.2
- net SENSE17_PRE: now also J28.1; no longer J27.1
- net SENSE18: now also DRIVE.R1.1, SENSE18.R1.2
- net THERM1: now also J19.1; no longer J21.1
- net THERM2: now also J20.1; no longer J22.1
- net THERM3: now also J21.1; no longer J23.1
- net THERM4: now also J22.1; no longer J24.1
- net THERM5: now also J23.1; no longer J25.1
- net THERM6: now also J24.1; no longer J26.1
- net V+: now also SENSE18.C1.1, SENSE18.R1.1; no longer C6.1, R3.2
- net V-: now also C6.1, C7.2, C8.1, CELL0.C1.2, CELL0.R1.1, DRIVE.C1.2, J19.2, J20.2, R1.1, SENSE18.C1.2; no longer C10.2, C4.2, C6.2, C7.1, C8.2, C9.1, J25.2, J26.2, R7.1, R9.1

Commit message: started placing ltc6813
Parts:
- C1, C2, C3: value (none) -> CAPACITOR_0603_10V_1UF
- C5, C6, C7, C8: value (none) -> CAPACITOR_0603_10V_10NF
- CELL0.C1, CELL10:C1, CELL11:C1, CELL12:C1, CELL13:C1, CELL14:C1, CELL15:C1, CELL16:C1, CELL17:C1, CELL18:C1, CELL1:C1, CELL2:C1, CELL3:C1, CELL4:C1, CELL5:C1, CELL6:C1, CELL7:C1, CELL8:C1, CELL9:C1, THERM1:C1, THERM2:C1, THERM3:C1, THERM4:C1, THERM5:C1, THERM6:C1, THERM7:C1, THERM8:C1, THERM9:C1: value (none) -> CAPACITOR_0603_100V_10NF
- DRIVE.C1, SENSE18.C1: value (none) -> CAPACITOR_0603_100V_0.1UF
- T1: value TRANSFORMERHM2102NLT -> TRANSFORMER
- moved R2 1059.2 mm to (120.9, -74.7), turned to 90 degrees
- moved R1 1057.6 mm to (122.4, -74.7), turned to 90 degrees
- moved C6 1050.8 mm to (138.4, -83.8)
- moved C8 1049.0 mm to (125.2, -80.6), turned to 180 degrees
- moved C7 1043.5 mm to (124.4, -83.8), turned to 270 degrees
- moved R6 1036.0 mm to (126.4, -83.8), turned to 270 degrees
- moved R5 1030.5 mm to (122.4, -83.8), turned to 270 degrees
- moved C5 1027.6 mm to (112.1, -86.4), turned to 90 degrees
- moved C3 1024.0 mm to (119.4, -74.7), turned to 270 degrees
- moved R4 1022.0 mm to (113.0, -82.5), turned to 90 degrees
- moved C2 1020.3 mm to (117.9, -74.7), turned to 270 degrees
- moved R3 1016.6 mm to (109.2, -82.5), turned to 90 degrees
- moved C1 1016.5 mm to (116.3, -74.7), turned to 270 degrees
- moved J17 1003.5 mm to (209.3, -33.5)
- moved J18 995.3 mm to (234.9, -77.5)
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Connections:
- net N$1 renamed ICMP
- net N$2 renamed IBIAS
- net N$25 renamed VREF1
- net IMA: now also T1.12; no longer T1.9
- net IMB: now also R5.2, T1.9; no longer R5.1, T1.12
- net IPA: now also T1.10; no longer T1.7
- net IPB: now also T1.7; no longer T1.10
- net ISO_IMA: now also T1.1; no longer T1.4
- net ISO_IMB: now also T1.4; no longer T1.1
- net ISO_IPA: now also T1.3; no longer T1.6
- net ISO_IPB: now also T1.6; no longer T1.3
- net N$18: now also C8.1, R5.1; no longer C8.2, R5.2
- net N$3: now also T1.11; no longer T1.8
- net N$4: now also C7.2, T1.8; no longer C7.1, T1.11
- net V-: now also C7.1, C8.2; no longer C7.2, C8.1
Routing:
- net V-: track 0.00 -> 31.4 mm
- net IMB: track 0.00 -> 16.8 mm
- net IPB: track 0.00 -> 16.4 mm
- net IPA: track 0.00 -> 10.9 mm
- net VREG: track 0.00 -> 9.36 mm
- net IMA: track 0.00 -> 8.77 mm
- net N$18: track 0.00 -> 8.68 mm
- net ICMP: track 0.00 -> 4.56 mm
- net VREF2: track 0.00 -> 3.12 mm
- net N$4: track 0.00 -> 2.52 mm
- net VREF1: track 0.00 -> 2.47 mm
- net IBIAS: track 0.00 -> 2.35 mm
Other:
- board size 108 x 240.3 mm -> 240.3 x 108 mm

Commit message: Last commit? :(
Parts:
- moved R1 1.52 mm to (120.9, -74.7)
- moved R2 1.52 mm to (122.4, -74.7)
Connections:
- net IBIAS: now also R1.2; no longer R2.2
- net ICMP: now also R1.1, R2.2; no longer R1.2, R2.1
- net V-: now also R2.1; no longer R1.1
Changed lines of the file:
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@@
 <attribute name="MOPN" value="603-CC603KRX7R6BB105" x="116.332" y="-74.676" size="1.778" layer="27" rot="R270" display="off"/>
 <attribute name="MPN" value="CC0603KRX7R6BB105" x="116.332" y="-74.676" size="1.778" layer="27" rot="R270" display="off"/>
-<attribute name="NAME" x="117.082" y="-74.676" size="0.8128" layer="25" font="vector" rot="R270" align="bottom-center"/>
+<attribute name="NAME" x="116.332" y="-76.2" size="0.8128" layer="25" font="vector" align="top-center"/>
 <attribute name="TOLERANCE" value="10%" x="116.332" y="-74.676" size="1.778" layer="27" rot="R270" display="off"/>
 <attribute name="VOLTAGE" value="10V" x="116.332" y="-74.676" size="1.778" layer="27" rot="R270" display="off"/>
@@
 <attribute name="MOPN" value="603-CC603KRX7R6BB105" x="117.856" y="-74.676" size="1.778" layer="27" rot="R270" display="off"/>
 <attribute name="MPN" value="CC0603KRX7R6BB105" x="117.856" y="-74.676" size="1.778" layer="27" rot="R270" display="off"/>
-<attribute name="NAME" x="118.606" y="-74.676" size="0.8128" layer="25" font="vector" rot="R270" align="bottom-center"/>
+<attribute name="NAME" x="117.856" y="-76.2" size="0.8128" layer="25" font="vector" align="top-center"/>
 <attribute name="TOLERANCE" value="10%" x="117.856" y="-74.676" size="1.778" layer="27" rot="R270" display="off"/>
 <attribute name="VOLTAGE" value="10V" x="117.856" y="-74.676" size="1.778" layer="27" rot="R270" display="off"/>
@@
 <attribute name="MOPN" value="603-CC603KRX7R6BB105" x="119.38" y="-74.676" size="1.778" layer="27" rot="R270" display="off"/>
 <attribute name="MPN" value="CC0603KRX7R6BB105" x="119.38" y="-74.676" size="1.778" layer="27" rot="R270" display="off"/>
-<attribute name="NAME" x="120.13" y="-74.676" size="0.8128" layer="25" font="vector" rot="R270" align="bottom-center"/>
+<attribute name="NAME" x="119.38" y="-76.2" size="0.8128" layer="25" font="vector" align="top-center"/>
 <attribute name="TOLERANCE" value="10%" x="119.38" y="-74.676" size="1.778" layer="27" rot="R270" display="off"/>
 <attribute name="VOLTAGE" value="10V" x="119.38" y="-74.676" size="1.778" layer="27" rot="R270" display="off"/>
@@
 <attribute name="VOLTAGE" value="100V" x="-615.95" y="-826.77" size="1.778" layer="27" display="off"/>
 </element>
-<element name="R1" library="HyTechDevices" package="0603-RES" value="RESISTOR_0603_1K" x="122.428" y="-74.676" smashed="yes" rot="R90">
+<element name="R2" library="HyTechDevices" package="0603-RES" value="RESISTOR_0603_1K" x="122.428" y="-74.676" smashed="yes" rot="R90">
 <attribute name="DKPN" value="311-1.00KHRCT-ND" x="122.428" y="-74.676" size="1.778" layer="27" rot="R90" display="off"/>
 <attribute name="MANUFACTURER" value="Yageo" x="122.428" y="-74.676" size="1.778" layer="27" rot="R90" display="off"/>
 <attribute name="MOPN" value="603-RC0603FR-071KL" x="122.428" y="-74.676" size="1.778" layer="27" rot="R90" display="off"/>
 <attribute name="MPN" value="RC0603FR-071KL" x="122.428" y="-74.676" size="1.778" layer="27" rot="R90" display="off"/>
-<attribute name="NAME" x="122.428" y="-76.2508" size="0.8128" layer="25" font="vector" align="top-center"/>
+<attribute name="NAME" x="122.428" y="-76.2" size="0.8128" layer="25" font="vector" align="top-center"/>
 <attribute name="POWER" value="0.1W" x="122.428" y="-74.676" size="1.778" layer="27" rot="R90" display="off"/>
 <attribute name="RESISTANCE" value="1k" x="122.428" y="-74.676" size="1.778" layer="27" rot="R90" display="off"/>
@@
 <attribute name="VOLTAGE" value="75V" x="122.428" y="-74.676" size="1.778" layer="27" rot="R90" display="off"/>
 </element>
-<element name="R2" library="HyTechDevices" package="0603-RES" value="RESISTOR_0603_1K" x="120.904" y="-74.676" smashed="yes" rot="R90">
+<element name="R1" library="HyTechDevices" package="0603-RES" value="RESISTOR_0603_1K" x="120.904" y="-74.676" smashed="yes" rot="R90">
 <attribute name="DKPN" value="311-1.00KHRCT-ND" x="120.904" y="-74.676" size="1.778" layer="27" rot="R90" display="off"/>
 <attribute name="MANUFACTURER" value="Yageo" x="120.904" y="-74.676" size="1.778" layer="27" rot="R90" display="off"/>
 <attribute name="MOPN" value="603-RC0603FR-071KL" x="120.904" y="-74.676" size="1.778" layer="27" rot="R90" display="off"/>
 <attribute name="MPN" value="RC0603FR-071KL" x="120.904" y="-74.676" size="1.778" layer="27" rot="R90" display="off"/>
-<attribute name="NAME" x="120.904" y="-76.2508" size="0.8128" layer="25" font="vector" align="top-center"/>
+<attribute name="NAME" x="120.904" y="-76.2" size="0.8128" layer="25" font="vector" align="top-center"/>
 <attribute name="POWER" value="0.1W" x="120.904" y="-74.676" size="1.778" layer="27" rot="R90" display="off"/>
 <attribute name="RESISTANCE" value="1k" x="120.904" y="-74.676" size="1.778" layer="27" rot="R90" display="off"/>
@@
 <signal name="ICMP">
 <contactref element="U1" pad="58"/>
-<contactref element="R1" pad="2"/>
-<contactref element="R2" pad="1"/>
+<contactref element="R2" pad="2"/>
+<contactref element="R1" pad="1"/>
 <wire x1="120.904" y1="-75.526" x2="122.4788" y2="-73.7734" width="0.254" layer="1"/>
 <wire x1="122.4788" y1="-73.7734" x2="122.428" y2="-73.826" width="0.254" layer="1"/>
@@
 <signal name="IBIAS">
 <contactref element="U1" pad="57"/>
-<contactref element="R2" pad="2"/>
+<contactref element="R1" pad="2"/>
 <wire x1="120.904" y1="-73.826" x2="121.662" y2="-73.068" width="0.254" layer="1"/>
 <wire x1="121.662" y1="-73.068" x2="121.662" y2="-71.79" width="0.254" layer="1"/>
@@
 <contactref element="C6" pad="1"/>
 <contactref element="SENSE18.C1" pad="2"/>
-<contactref element="R1" pad="1"/>
+<contactref element="R2" pad="1"/>
 <contactref element="C7" pad="1"/>
 <contactref element="C8" pad="2"/>
