File: EAGLE Board Designs/BMS/BMS Segment/BMS Segment rev15 new.brd (EAGLE design)
At the start: 108 x 240.3 mm, 294 parts, among them J1_A 0R, J1_B 0R, J2_A 0R, J2_B 0R, J3_A 0R, J3_B 0R, J4_A 0R, J4_B 0R, J5_A 0R, J5_B 0R, J6_A 0R, J6_B 0R, J7_A 0R, J7_B 0R, J8_A 0R, J8_B 0R, Q1 NSV1C201MZ4, Q2 NSV1C201MZ4, U1 LTC6811-2, U2 LTC6811-2

Commit message: Replaced fuses and resistors
Parts:
- DRAIN10:DISCHARGE, DRAIN11:DISCHARGE, DRAIN12:DISCHARGE, DRAIN13:DISCHARGE, DRAIN14:DISCHARGE, DRAIN15:DISCHARGE, DRAIN16:DISCHARGE, DRAIN17:DISCHARGE, DRAIN18:DISCHARGE, DRAIN1:DISCHARGE, DRAIN2:DISCHARGE, DRAIN3:DISCHARGE, DRAIN4:DISCHARGE, DRAIN5:DISCHARGE, DRAIN6:DISCHARGE, DRAIN7:DISCHARGE, DRAIN8:DISCHARGE, DRAIN9:DISCHARGE: value 5R -> RESISTOR_PWR263_; device HyTechDevices:PWR163 -> HyTechDevices:PWR263
- DRAIN10:GATE, DRAIN10:R, DRAIN10:R1, DRAIN11:GATE, DRAIN11:R, DRAIN11:R1, DRAIN12:GATE, DRAIN12:R, DRAIN12:R1, DRAIN13:GATE, DRAIN13:R, DRAIN13:R1, DRAIN14:GATE, DRAIN14:R, DRAIN14:R1, DRAIN15:GATE, DRAIN15:R, DRAIN15:R1, DRAIN16:GATE, DRAIN16:R, DRAIN16:R1, DRAIN17:GATE, DRAIN17:R, DRAIN17:R1, DRAIN18:GATE, DRAIN18:R, DRAIN18:R1, DRAIN1:GATE, DRAIN1:R, DRAIN1:R1, DRAIN2:GATE, DRAIN2:R, DRAIN2:R1, DRAIN3:GATE, DRAIN3:R, DRAIN3:R1, DRAIN4:GATE, DRAIN4:R, DRAIN4:R1, DRAIN5:GATE, DRAIN5:R, DRAIN5:R1, DRAIN6:GATE, DRAIN6:R, DRAIN6:R1, DRAIN7:GATE, DRAIN7:R, DRAIN7:R1, DRAIN8:GATE, DRAIN8:R, DRAIN8:R1, DRAIN9:GATE, DRAIN9:R, DRAIN9:R1, J1_A, J1_B, J2_A, J2_B, J3_A, J3_B, J4_A, J4_B, J5_A, J5_B, J6_A, J6_B, J7_A, J7_B, J8_A, J8_B, J_CELL_A, J_THERM_A, R1_A, R1_B, R2_A, R2_B, R3_A, R3_B, R4_A, R4_B, R5_A, R5_B, RB1_A, RB1_B, RB2_A, RB2_B, RIN_A, RIN_B, RM_A, RM_B, RU1_A, RU1_B, RU2_A, RU2_B, THERM_FILTER10:R, THERM_FILTER10:R1, THERM_FILTER1:R, THERM_FILTER1:R1, THERM_FILTER2:R, THERM_FILTER2:R1, THERM_FILTER3:R, THERM_FILTER3:R1, THERM_FILTER4:R, THERM_FILTER4:R1, THERM_FILTER5:R, THERM_FILTER5:R1, THERM_FILTER6:R, THERM_FILTER6:R1, THERM_FILTER7:R, THERM_FILTER7:R1, THERM_FILTER8:R, THERM_FILTER8:R1, THERM_FILTER9:R, THERM_FILTER9:R1: device HyTechDevices:0603-RES -> HyTechDevices:0603-RES@1
- F0, F1, F10, F11, F12, F13, F14, F15, F16, F17, F18, F2, F3, F4, F5, F6, F7, F8, F9: device HyTechDevices:5X20MM_FUSE -> HyTechDevices:0885
- moved U$29 15.1 mm to (82.4, 67.4), turned to 90 degrees
- moved CELL17 14.1 mm to (38.2, 222.6)
- moved DRAIN4:DISCHARGE 12.8 mm to (80.3, 52.6)
- moved CELL15 12.5 mm to (38.2, 196.3)
- moved DRAIN8:DISCHARGE 12.3 mm to (80.3, 105.4)
- moved DRAIN18:DISCHARGE 12.1 mm to (83.4, 235.6)
- moved DRAIN14:DISCHARGE 11.9 mm to (80.3, 185.0)
- moved DRAIN6:DISCHARGE 11.5 mm to (77.6, 77.9)
- moved CELL13 11.4 mm to (38.2, 170.4)
- moved DRAIN16:DISCHARGE 11.4 mm to (80.3, 211.1)
- moved DRAIN12:DISCHARGE 11.1 mm to (80.3, 157.5)
- moved DRAIN10:DISCHARGE 11.0 mm to (80.3, 130.8)
- moved DRAIN2:DISCHARGE 10.9 mm to (80.3, 26.0)
- moved CELL11 9.22 mm to (38.2, 143.3)
- moved DRAIN11:DISCHARGE 9.18 mm to (26.0, 134.6)
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Connections:
- net CC0: now also F0.1; no longer F0.P$1
- net CC1: now also F1.1; no longer F1.P$1
- net CC10: now also F10.1; no longer F10.P$1
- net CC11: now also F11.1; no longer F11.P$1
- net CC12: now also F12.1; no longer F12.P$1
- net CC13: now also F13.1; no longer F13.P$1
- net CC14: now also F14.1; no longer F14.P$1
- net CC15: now also F15.1; no longer F15.P$1
- net CC16: now also F16.1; no longer F16.P$1
- net CC17: now also F17.1; no longer F17.P$1
- net CC18: now also F18.1; no longer F18.P$1
- net CC2: now also F2.1; no longer F2.P$1
- net CC3: now also F3.1; no longer F3.P$1
- net CC4: now also F4.1; no longer F4.P$1
- net CC5: now also F5.1; no longer F5.P$1
- net CC6: now also F6.1; no longer F6.P$1
- net CC7: now also F7.1; no longer F7.P$1
- net CC8: now also F8.1; no longer F8.P$1
- net CC9: now also F9.1; no longer F9.P$1
- net SENSE1: now also F1.2; no longer F1.P$2
- net SENSE10: now also F10.2; no longer F10.P$2
- net SENSE11: now also F11.2; no longer F11.P$2
- net SENSE12: now also F12.2; no longer F12.P$2
- net SENSE13: now also F13.2; no longer F13.P$2
- net SENSE14: now also F14.2; no longer F14.P$2
- net SENSE15: now also F15.2; no longer F15.P$2
- net SENSE16: now also F16.2; no longer F16.P$2
- net SENSE17_PRE: now also F17.2; no longer F17.P$2
- net SENSE18: now also F18.2; no longer F18.P$2
- net SENSE2: now also F2.2; no longer F2.P$2
- net SENSE3: now also F3.2; no longer F3.P$2
- net SENSE4: now also F4.2; no longer F4.P$2
- net SENSE5: now also F5.2; no longer F5.P$2
- net SENSE6: now also F6.2; no longer F6.P$2
- net SENSE7: now also F7.2; no longer F7.P$2
- net SENSE8: now also F8.2; no longer F8.P$2
- net V-_A: now also F9.2; no longer F9.P$2
- net V-_B: now also F0.2; no longer F0.P$2
Routing:
- net DRAIN18:N$1: track 11.3 -> 19.3 mm
- net V-_A: track 816.5 -> 824.4 mm, vias 29 -> 31
- net CC17: track 25.8 -> 18.5 mm
- net CC13: track 26.8 -> 19.9 mm
- net S10_A: track 60.2 -> 67.0 mm
- net DRAIN8:N$1: track 10.7 -> 16.4 mm
- net DRAIN2:N$1: track 12.0 -> 17.4 mm
- net DRAIN10:N$1: track 14.9 -> 20.2 mm
- net CC2: track 23.3 -> 28.6 mm
- net SENSE18: track 161.1 -> 155.8 mm
- net SENSE7: track 61.5 -> 66.6 mm
- net DRAIN18:GATE: track 8.45 -> 3.27 mm
- net SENSE6: track 58.7 -> 53.6 mm
- net C7_B: track 38.8 -> 43.8 mm
- net CC18: track 25.1 -> 20.2 mm
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