File: EAGLE Board Designs/Testing and Practice Boards/Testing Boards/Power Switching Circuit rev1 - old.sch (EAGLE design)
At the start: 47 parts, among them K1 J115F11A6, Q1 SIR638ADP, Q2 SIR638ADP, Q3 SIR638ADP, Q4 SIR638ADP, U1 LTC4421, X1 CONNECTOR-4AUTOSPORT, X2 CONNECTOR-4AUTOSPORT, X3 CONNECTOR-3

Commit message: Ethan's updates
Parts:
- removed D1, D2: SCHOTTKY, HyTechDevices:SCHOTTKY
- removed RN1, RN2: RESISTOR_NETWORK_4_10K, HyTechDevices:RESISTOR_NETWORK_4_10K
- added D3, D4: DIODEREMOVE_IN_XML, HyTechDevices:DIODEREMOVE_IN_XML
- added R10, R5, R6, R7, R8, R9: 100k, HyTechDevices:RESISTOR0603
- renumbered D5 to TVS2, D6 to TVS, K1 to RELAY, Q1 to U$4, Q2 to U$5, Q3 to U$6, Q4 to U$7, U1 to LTC4421
Connections:
- net !SHDN: now also D3.C, D4.C; no longer D1.C, D2.C
- net CASIN: now also R10.2, R5.2, R6.2, R7.2, R8.2, R9.2; no longer RN1A.2, RN1B.2, RN1C.2, RN1D.2, RN2C.2, RN2D.2
- net GLVMS: now also D4.A; no longer D2.A
- net N$11: now also R5.1; no longer RN1D.1
- net N$13: now also R6.1; no longer RN1C.1
- net N$15: now also R7.1; no longer RN1B.1
- net N$17: now also R8.1; no longer RN1A.1
- net N$19: now also R9.1; no longer RN2D.1
- net N$21: now also R10.1; no longer RN2C.1
- net START: now also D3.A; no longer D1.A
